File: kbms.sch (KiCad schematic (older format))
At the start: 12 parts, among them J12 AVR-ISP-6, J13 DE9 Male, J14 DE9 Male, J15 Mini-DIN-6, J16 Mini-DIN-6, U6 ATmega328-PU

Commit message: Replace two PS/2 headers with single double-header.
Parts:
- removed J15, J16: Mini-DIN-6, JGP Footprints:mini-DIN 6, symbol Connector:Mini-DIN-6
- added J15: Double-mini-DIN-6, symbol ExtraConnectors:Double-mini-DIN-6
Changed lines of the file:
@@
 Text HLabel 4400 4300 2    50   Output ~ 0
 KBMS_TO_MCU
-$Comp
-L Connector:Mini-DIN-6 J?
-U 1 1 5DF4AE86
-P 9700 3150
-AR Path="/5DF4AE86" Ref="J?"  Part="1"
-AR Path="/5DF2662E/5DF4AE86" Ref="J15"  Part="1"
-F 0 "J15" H 9700 3517 50  0000 C CNN
-F 1 "Mini-DIN-6" H 9700 3426 50  0000 C CNN
-F 2 "JGP Footprints:mini-DIN 6" H 9700 3150 50  0001 C CNN
-F 3 "http://service.powerdynamics.com/ec/Catalog17/Section%2011.pdf" H 9700 3150 50  0001 C CNN
-	1    9700 3150
-	1    0    0    -1
-$EndComp
-$Comp
-L Connector:Mini-DIN-6 J?
-U 1 1 5DF4AE8C
-P 9700 3950
-AR Path="/5DF4AE8C" Ref="J?"  Part="1"
-AR Path="/5DF2662E/5DF4AE8C" Ref="J16"  Part="1"
-F 0 "J16" H 9700 4317 50  0000 C CNN
-F 1 "Mini-DIN-6" H 9700 4226 50  0000 C CNN
-F 2 "JGP Footprints:mini-DIN 6" H 9700 3950 50  0001 C CNN
-F 3 "http://service.powerdynamics.com/ec/Catalog17/Section%2011.pdf" H 9700 3950 50  0001 C CNN
-	1    9700 3950
-	1    0    0    -1
-$EndComp
 Text HLabel 4800 4200 2    50   Input ~ 0
 ~RESET
@@
 L power:+5V #PWR?
 U 1 1 5E1B9008
-P 9200 2850
+P 9350 3450
 AR Path="/5E1B9008" Ref="#PWR?"  Part="1"
 AR Path="/5DF2662E/5E1B9008" Ref="#PWR?"  Part="1"
-F 0 "#PWR?" H 9200 2700 50  0001 C CNN
-F 1 "+5V" H 9215 3023 50  0000 C CNN
-F 2 "" H 9200 2850 50  0001 C CNN
-F 3 "" H 9200 2850 50  0001 C CNN
-	1    9200 2850
-	1    0    0    -1
-$EndComp
-Wire Wire Line
-	9400 3150 9200 3150
-Wire Wire Line
-	9200 3150 9200 2850
-Wire Wire Line
-	9200 3950 9200 3150
-Connection ~ 9200 3150
-NoConn ~ 9400 3050
-NoConn ~ 9400 3250
-NoConn ~ 9400 3850
-NoConn ~ 9400 4050
-Wire Wire Line
-	9200 3950 9400 3950
+F 0 "#PWR?" H 9350 3300 50  0001 C CNN
+F 1 "+5V" H 9365 3623 50  0000 C CNN
+F 2 "" H 9350 3450 50  0001 C CNN
+F 3 "" H 9350 3450 50  0001 C CNN
+	1    9350 3450
+	1    0    0    -1
+$EndComp
+Wire Wire Line
+	9550 3750 9350 3750
+Wire Wire Line
+	9350 3750 9350 3450
+Connection ~ 9350 3750
+NoConn ~ 9550 3650
+NoConn ~ 9550 3850
+NoConn ~ 9550 4200
+NoConn ~ 9550 4400
 $Comp
 L power:GND #PWR?
 U 1 1 5E1BC21F
-P 10150 4200
+P 10300 4550
 AR Path="/5E1BC21F" Ref="#PWR?"  Part="1"
 AR Path="/5DF2662E/5E1BC21F" Ref="#PWR?"  Part="1"
-F 0 "#PWR?" H 10150 3950 50  0001 C CNN
-F 1 "GND" H 10155 4027 50  0000 C CNN
-F 2 "" H 10150 4200 50  0001 C CNN
-F 3 "" H 10150 4200 50  0001 C CNN
-	1    10150 4200
-	1    0    0    -1
-$EndComp
-Wire Wire Line
-	10000 3150 10150 3150
-Wire Wire Line
-	10150 3150 10150 3950
-Wire Wire Line
-	10000 3950 10150 3950
-Connection ~ 10150 3950
-Wire Wire Line
-	10150 3950 10150 4200
-Text Label 10250 3050 0    50   ~ 0
+F 0 "#PWR?" H 10300 4300 50  0001 C CNN
+F 1 "GND" H 10305 4377 50  0000 C CNN
+F 2 "" H 10300 4550 50  0001 C CNN
+F 3 "" H 10300 4550 50  0001 C CNN
+	1    10300 4550
+	1    0    0    -1
+$EndComp
+Wire Wire Line
+	10150 3750 10300 3750
+Wire Wire Line
+	10150 4300 10300 4300
+Connection ~ 10300 4300
+Wire Wire Line
+	10300 4300 10300 4550
+Text Label 10400 3650 0    50   ~ 0
 KB_CLK
-Text Label 10250 3250 0    50   ~ 0
+Text Label 10400 3850 0    50   ~ 0
 KB_DAT
-Text Label 10250 3850 0    50   ~ 0
+Text Label 10400 4200 0    50   ~ 0
 MS_CLK
-Text Label 10250 4050 0    50   ~ 0
+Text Label 10400 4400 0    50   ~ 0
 MS_DAT
 Wire Wire Line
-	10000 3050 10500 3050
-Wire Wire Line
-	10000 3250 10500 3250
-Wire Wire Line
-	10000 3850 10500 3850
-Wire Wire Line
-	10000 4050 10500 4050
+	10150 3650 10650 3650
+Wire Wire Line
+	10150 3850 10650 3850
+Wire Wire Line
+	10150 4200 10650 4200
+Wire Wire Line
+	10150 4400 10650 4400
 $Comp
 L Connector:DB9_Male J?
@@
 Wire Wire Line
 	3200 1700 3400 1700
+$Comp
+L ExtraConnectors:Double-mini-DIN-6 J15
+U 1 1 5E0028E3
+P 9850 4000
+F 0 "J15" H 9850 4698 50  0000 C CNN
+F 1 "Double-mini-DIN-6" H 9850 4607 50  0000 C CNN
+F 2 "" H 9850 4250 50  0001 C CNN
+F 3 "http://www.mouser.com/ds/2/18/40_c091_abd_e-75918.pdf" H 9850 4250 50  0001 C CNN
+	1    9850 4000
+	1    0    0    -1
+$EndComp
+Wire Wire Line
+	10300 3750 10300 4300
+Wire Wire Line
+	9550 4300 9350 4300
+Wire Wire Line
+	9350 4300 9350 3750
 $EndSCHEMATC

Commit message: Replaced keyboard/mouse connect with double PS/2 header.
Jiggled around PCB layout to line more tracks up on grid.
Parts:
- J15: footprint (none) -> JGP Footprints:Double_mini-DIN_6
Changed lines of the file:
@@
 F 0 "J15" H 9850 4698 50  0000 C CNN
 F 1 "Double-mini-DIN-6" H 9850 4607 50  0000 C CNN
-F 2 "" H 9850 4250 50  0001 C CNN
+F 2 "JGP Footprints:Double_mini-DIN_6" H 9850 4250 50  0001 C CNN
 F 3 "http://www.mouser.com/ds/2/18/40_c091_abd_e-75918.pdf" H 9850 4250 50  0001 C CNN
 	1    9850 4000

Commit message: Adding MPNs.
Parts:
- J12: Manufacturer (none) -> Harwin; PartNo (none) -> M20-9980346
- J13, J14: footprint Connector_Dsub:DSUB-9_Female_Horizontal_P2.77x2.84mm_EdgePinOffset4.94mm_Housed_MountingHolesOffset7.48mm -> Connector_Dsub:DSUB-9_Male_Horizontal_P2.77x2.84mm_EdgePinOffset4.94mm_Housed_MountingHolesOffset7.48mm
- J15: Manufacturer (none) -> Kycon; PartNo (none) -> KMDGX-6S-6S-S4N.
- R19, R20, R21: Manufacturer (none) -> Stackpole Electronics Inc; PartNo (none) -> CF14JT1K00R
- U6: Manufacturer (none) -> Microchip; PartNo (none) -> ATmega328-PU
Changed lines of the file:
@@
 F 0 "J13" H 8730 3402 50  0000 L CNN
 F 1 "DE9 Male" H 8730 3311 50  0000 L CNN
-F 2 "Connector_Dsub:DSUB-9_Female_Horizontal_P2.77x2.84mm_EdgePinOffset4.94mm_Housed_MountingHolesOffset7.48mm" H 8550 3400 50  0001 C CNN
+F 2 "Connector_Dsub:DSUB-9_Male_Horizontal_P2.77x2.84mm_EdgePinOffset4.94mm_Housed_MountingHolesOffset7.48mm" H 8550 3400 50  0001 C CNN
 F 3 " ~" H 8550 3400 50  0001 C CNN
 	1    8550 3400
@@
 F 0 "J14" H 8730 4802 50  0000 L CNN
 F 1 "DE9 Male" H 8730 4711 50  0000 L CNN
-F 2 "Connector_Dsub:DSUB-9_Female_Horizontal_P2.77x2.84mm_EdgePinOffset4.94mm_Housed_MountingHolesOffset7.48mm" H 8550 4800 50  0001 C CNN
+F 2 "Connector_Dsub:DSUB-9_Male_Horizontal_P2.77x2.84mm_EdgePinOffset4.94mm_Housed_MountingHolesOffset7.48mm" H 8550 4800 50  0001 C CNN
 F 3 " ~" H 8550 4800 50  0001 C CNN
 	1    8550 4800
@@
 F 2 "Resistor_THT:R_Axial_DIN0207_L6.3mm_D2.5mm_P10.16mm_Horizontal" V 5180 3250 50  0001 C CNN
 F 3 "~" H 5250 3250 50  0001 C CNN
+F 4 "Stackpole Electronics Inc" H 5250 3250 50  0001 C CNN "Manufacturer"
+F 5 "CF14JT1K00R" H 5250 3250 50  0001 C CNN "PartNo"
 	1    5250 3250
 	0    1    1    0
@@
 F 2 "Resistor_THT:R_Axial_DIN0207_L6.3mm_D2.5mm_P10.16mm_Horizontal" V 5180 3400 50  0001 C CNN
 F 3 "~" H 5250 3400 50  0001 C CNN
+F 4 "Stackpole Electronics Inc" H 5250 3400 50  0001 C CNN "Manufacturer"
+F 5 "CF14JT1K00R" H 5250 3400 50  0001 C CNN "PartNo"
 	1    5250 3400
 	0    1    1    0
@@
 F 2 "Resistor_THT:R_Axial_DIN0207_L6.3mm_D2.5mm_P10.16mm_Horizontal" V 5180 3550 50  0001 C CNN
 F 3 "~" H 5250 3550 50  0001 C CNN
+F 4 "Stackpole Electronics Inc" H 5250 3550 50  0001 C CNN "Manufacturer"
+F 5 "CF14JT1K00R" H 5250 3550 50  0001 C CNN "PartNo"
 	1    5250 3550
 	0    1    1    0
@@
 F 2 "Connector_PinHeader_2.54mm:PinHeader_2x03_P2.54mm_Vertical" V 6600 2300 50  0001 C CNN
 F 3 " ~" H 5575 1700 50  0001 C CNN
+F 4 "Harwin" H 6850 2250 50  0001 C CNN "Manufacturer"
+F 5 "M20-9980346" H 6850 2250 50  0001 C CNN "PartNo"
 	1    6850 2250
 	-1   0    0    -1
@@
 F 2 "Package_DIP:DIP-28_W7.62mm" H 3100 3800 50  0001 C CIN
 F 3 "http://ww1.microchip.com/downloads/en/DeviceDoc/ATmega328_P%20AVR%20MCU%20with%20picoPower%20Technology%20Data%20Sheet%2040001984A.pdf" H 3100 3800 50  0001 C CNN
+F 4 "Microchip" H 3100 3800 50  0001 C CNN "Manufacturer"
+F 5 "ATmega328-PU" H 3100 3800 50  0001 C CNN "PartNo"
 	1    3100 3800
 	1    0    0    -1
@@
 F 1 "Double-mini-DIN-6" H 9850 4607 50  0000 C CNN
 F 2 "JGP Footprints:Double_mini-DIN_6" H 9850 4250 50  0001 C CNN
-F 3 "http://www.mouser.com/ds/2/18/40_c091_abd_e-75918.pdf" H 9850 4250 50  0001 C CNN
+F 3 "http://www.kycon.com/Pub_Eng_Draw/KMDGX-6S-6S-S4N.pdf" H 9850 4250 50  0001 C CNN
+F 4 "Kycon" H 9850 4000 50  0001 C CNN "Manufacturer"
+F 5 "KMDGX-6S-6S-S4N." H 9850 4000 50  0001 C CNN "PartNo"
 	1    9850 4000
 	1    0    0    -1

Commit message: Use offset DE9 for Joysticks.
Parts:
- J12: symbol Connector:AVR-ISP-6 -> neotron-32-rescue:AVR-ISP-6-Connector
- J13, J14: footprint Connector_Dsub:DSUB-9_Male_Horizontal_P2.77x2.84mm_EdgePinOffset4.94mm_Housed_MountingHolesOffset7.48mm -> Connector_Dsub:DSUB-9_Male_Horizontal_P2.77x2.84mm_EdgePinOffset14.56mm_Housed_MountingHolesOffset8.20mm; Manufacturer (none) -> TE; PartNo (none) -> 5747467-2
- J15: symbol ExtraConnectors:Double-mini-DIN-6 -> neotron-32-rescue:Double-mini-DIN-6-ExtraConnectors
- U6: symbol MCU_Microchip_ATmega:ATmega328-PU -> neotron-32-rescue:ATmega328-PU-MCU_Microchip_ATmega
Changed lines of the file:
@@
 EESchema Schematic File Version 4
-EELAYER 30 0
+LIBS:neotron-32-cache
+EELAYER 26 0
 EELAYER END
 $Descr A4 11693 8268
@@
 F 0 "J13" H 8730 3402 50  0000 L CNN
 F 1 "DE9 Male" H 8730 3311 50  0000 L CNN
-F 2 "Connector_Dsub:DSUB-9_Male_Horizontal_P2.77x2.84mm_EdgePinOffset4.94mm_Housed_MountingHolesOffset7.48mm" H 8550 3400 50  0001 C CNN
+F 2 "Connector_Dsub:DSUB-9_Male_Horizontal_P2.77x2.84mm_EdgePinOffset14.56mm_Housed_MountingHolesOffset8.20mm" H 8550 3400 50  0001 C CNN
 F 3 " ~" H 8550 3400 50  0001 C CNN
+F 4 "TE" H 0   0   50  0001 C CNN "Manufacturer"
+F 5 "5747467-2" H 0   0   50  0001 C CNN "PartNo"
 	1    8550 3400
 	1    0    0    -1
@@
 F 0 "J14" H 8730 4802 50  0000 L CNN
 F 1 "DE9 Male" H 8730 4711 50  0000 L CNN
-F 2 "Connector_Dsub:DSUB-9_Male_Horizontal_P2.77x2.84mm_EdgePinOffset4.94mm_Housed_MountingHolesOffset7.48mm" H 8550 4800 50  0001 C CNN
+F 2 "Connector_Dsub:DSUB-9_Male_Horizontal_P2.77x2.84mm_EdgePinOffset14.56mm_Housed_MountingHolesOffset8.20mm" H 8550 4800 50  0001 C CNN
 F 3 " ~" H 8550 4800 50  0001 C CNN
+F 4 "TE" H 0   0   50  0001 C CNN "Manufacturer"
+F 5 "5747467-2" H 0   0   50  0001 C CNN "PartNo"
 	1    8550 4800
 	1    0    0    -1
@@
 	3700 2800 5700 2800
 $Comp
-L Connector:AVR-ISP-6 J12
+L neotron-32-rescue:AVR-ISP-6-Connector J12
 U 1 1 5DF8E8EA
 P 6850 2250
+AR Path="/5DF8E8EA" Ref="J12"  Part="1"
+AR Path="/5DF2662E/5DF8E8EA" Ref="J12"  Part="1"
 F 0 "J12" H 6520 2346 50  0000 R CNN
 F 1 "AVR-ISP-6" H 6520 2255 50  0000 R CNN
@@
 	2700 1700 2550 1700
 $Comp
-L MCU_Microchip_ATmega:ATmega328-PU U6
+L neotron-32-rescue:ATmega328-PU-MCU_Microchip_ATmega U6
 U 1 1 5E0F9E16
 P 3100 3800
+AR Path="/5E0F9E16" Ref="U6"  Part="1"
+AR Path="/5DF2662E/5E0F9E16" Ref="U6"  Part="1"
 F 0 "U6" H 2456 3846 50  0000 R CNN
 F 1 "ATmega328-PU" H 2456 3755 50  0000 R CNN
@@
 	3200 1700 3400 1700
 $Comp
-L ExtraConnectors:Double-mini-DIN-6 J15
+L neotron-32-rescue:Double-mini-DIN-6-ExtraConnectors J15
 U 1 1 5E0028E3
 P 9850 4000
+AR Path="/5E0028E3" Ref="J15"  Part="1"
+AR Path="/5DF2662E/5E0028E3" Ref="J15"  Part="1"
 F 0 "J15" H 9850 4698 50  0000 C CNN
 F 1 "Double-mini-DIN-6" H 9850 4607 50  0000 C CNN

Commit message: Updated BOM.
Parts:
- C19, C20, C29: Manufacturer (none) -> Vishay; PartNo (none) -> K104K15X7RF5TL2
- J12: Manufacturer Harwin -> (none); PartNo M20-9980346 -> (none)
Changed lines of the file:
@@
 F 1 "DE9 Male" H 8730 3311 50  0000 L CNN
 F 2 "Connector_Dsub:DSUB-9_Male_Horizontal_P2.77x2.84mm_EdgePinOffset14.56mm_Housed_MountingHolesOffset8.20mm" H 8550 3400 50  0001 C CNN
-F 3 " ~" H 8550 3400 50  0001 C CNN
+F 3 "https://www.te.com/commerce/DocumentDelivery/DDEController?Action=srchrtrv&DocNm=5747467&DocType=Customer+Drawing&DocLang=English" H 8550 3400 50  0001 C CNN
 F 4 "TE" H 0   0   50  0001 C CNN "Manufacturer"
 F 5 "5747467-2" H 0   0   50  0001 C CNN "PartNo"
@@
 F 1 "DE9 Male" H 8730 4711 50  0000 L CNN
 F 2 "Connector_Dsub:DSUB-9_Male_Horizontal_P2.77x2.84mm_EdgePinOffset14.56mm_Housed_MountingHolesOffset8.20mm" H 8550 4800 50  0001 C CNN
-F 3 " ~" H 8550 4800 50  0001 C CNN
+F 3 "https://www.te.com/commerce/DocumentDelivery/DDEController?Action=srchrtrv&DocNm=5747467&DocType=Customer+Drawing&DocLang=English" H 8550 4800 50  0001 C CNN
 F 4 "TE" H 0   0   50  0001 C CNN "Manufacturer"
 F 5 "5747467-2" H 0   0   50  0001 C CNN "PartNo"
@@
 F 2 "Capacitor_THT:C_Disc_D3.0mm_W2.0mm_P2.50mm" H 2738 1700 50  0001 C CNN
 F 3 "~" H 2700 1850 50  0001 C CNN
+F 4 "Vishay" H 0   0   50  0001 C CNN "Manufacturer"
+F 5 "K104K15X7RF5TL2" H 0   0   50  0001 C CNN "PartNo"
 	1    2700 1850
 	1    0    0    -1
@@
 F 2 "Capacitor_THT:C_Disc_D3.0mm_W2.0mm_P2.50mm" H 2238 2650 50  0001 C CNN
 F 3 "~" H 2200 2800 50  0001 C CNN
+F 4 "Vishay" H 0   0   50  0001 C CNN "Manufacturer"
+F 5 "K104K15X7RF5TL2" H 0   0   50  0001 C CNN "PartNo"
 	1    2200 2800
 	1    0    0    1
@@
 F 1 "AVR-ISP-6" H 6520 2255 50  0000 R CNN
 F 2 "Connector_PinHeader_2.54mm:PinHeader_2x03_P2.54mm_Vertical" V 6600 2300 50  0001 C CNN
-F 3 " ~" H 5575 1700 50  0001 C CNN
-F 4 "Harwin" H 6850 2250 50  0001 C CNN "Manufacturer"
-F 5 "M20-9980346" H 6850 2250 50  0001 C CNN "PartNo"
+F 3 "~" H 5575 1700 50  0001 C CNN
+F 4 "~" H 6850 2250 50  0001 C CNN "Manufacturer"
+F 5 "~" H 6850 2250 50  0001 C CNN "PartNo"
 	1    6850 2250
 	-1   0    0    -1
@@
 F 2 "Capacitor_THT:C_Disc_D3.0mm_W2.0mm_P2.50mm" H 3438 1700 50  0001 C CNN
 F 3 "~" H 3400 1850 50  0001 C CNN
+F 4 "Vishay" H 0   0   50  0001 C CNN "Manufacturer"
+F 5 "K104K15X7RF5TL2" H 0   0   50  0001 C CNN "PartNo"
 	1    3400 1850
 	1    0    0    -1

Commit message: Add some extra explanatory notes.
Other:
- note added: "The AtMega 328 acts as the interface to the 5V PS/2 Keyboard and PS/2 Mouse, as well as the two 9-pin Joysticks. It buffers incoming\nevents and sends the buffered data in response to commands received over the UART. It can also activate the Keyboard LEDs and\nconfigure the Mouse sample rate.\n\nBoth Atari-compatible 9-pin joysticks and SEGA MegaDrive/Genesis 9-pin controllers are supported. The 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"
- note removed: "Keyboard, Mouse & Joystick"
Changed lines of the file:
@@
 EESchema Schematic File Version 4
-LIBS:neotron-32-cache
-EELAYER 26 0
+EELAYER 30 0
 EELAYER END
 $Descr A4 11693 8268
@@
 Wire Wire Line
 	5700 3100 8250 3100
-Text Notes 4450 1050 0    100  ~ 20
-Keyboard, Mouse & Joystick
 $Comp
 L Device:C C?
@@
 Wire Wire Line
 	9350 4300 9350 3750
+Text Notes 550  7700 0    50   Italic 0
+The AtMega 328 acts as the interface to the 5V PS/2 Keyboard and PS/2 Mouse, as well as the two 9-pin Joysticks. It buffers incoming\nevents and sends the buffered data in response to commands received over the UART. It can also activate the Keyboard LEDs and\nconfigure the Mouse sample rate.\n\nBoth Atari-compatible 9-pin joysticks and SEGA MegaDrive/Genesis 9-pin controllers are supported. The latter are detected when both\nLeft and Right are active (low); the AtMega will then flip the select line and read the 'other' set of pins.\n\nThe AtMega can be programmed via the standard ISP socket. Note that activating the AtMega AT_RESET line will reset the entire board.
 $EndSCHEMATC

Commit message: Fix Stackpole 1K part number.
Parts:
- R19, R20, R21: PartNo CF14JT1K00R -> CF14JT1K00
Changed lines of the file:
@@
 F 3 "~" H 5250 3250 50  0001 C CNN
 F 4 "Stackpole Electronics Inc" H 5250 3250 50  0001 C CNN "Manufacturer"
-F 5 "CF14JT1K00R" H 5250 3250 50  0001 C CNN "PartNo"
+F 5 "CF14JT1K00" H 5250 3250 50  0001 C CNN "PartNo"
 	1    5250 3250
 	0    1    1    0
@@
 F 3 "~" H 5250 3400 50  0001 C CNN
 F 4 "Stackpole Electronics Inc" H 5250 3400 50  0001 C CNN "Manufacturer"
-F 5 "CF14JT1K00R" H 5250 3400 50  0001 C CNN "PartNo"
+F 5 "CF14JT1K00" H 5250 3400 50  0001 C CNN "PartNo"
 	1    5250 3400
 	0    1    1    0
@@
 F 3 "~" H 5250 3550 50  0001 C CNN
 F 4 "Stackpole Electronics Inc" H 5250 3550 50  0001 C CNN "Manufacturer"
-F 5 "CF14JT1K00R" H 5250 3550 50  0001 C CNN "PartNo"
+F 5 "CF14JT1K00" H 5250 3550 50  0001 C CNN "PartNo"
 	1    5250 3550
 	0    1    1    0
