File: kbms.sch (KiCad schematic (older format))
At the start: 11 parts, among them J12 AVR-ISP-6, J13 DE9 Male, J14 DE9 Male, J15 Double-mini-DIN-6, U6 ATmega328-PU

Commit message: Tweaks to the BOM.
Marking parts as DNP=1 should stop them appearing in the BOM.
Also set multi-parts for ICs in sockets.
Parts:
- C19, C20, C29, J13, J14, J15, R19, R20, R21: DNP (none) -> 0
- J12: DNP (none) -> 0; Manufacturer (none) -> Harwin; mpn (none) -> M20-9760346
- U6: DNP (none) -> 0; Manufacturer Microchip -> Microchip;On Shore Technology; mpn ATmega328-PU -> ATmega328-PU;ED281DT
Changed lines of the file:
@@
 F 4 "TE" H 0   0   50  0001 C CNN "Manufacturer"
 F 5 "5747467-2" H 0   0   50  0001 C CNN "mpn"
+F 6 "0" H 8550 3400 50  0001 C CNN "DNP"
 	1    8550 3400
 	1    0    0    -1
@@
 F 4 "TE" H 0   0   50  0001 C CNN "Manufacturer"
 F 5 "5747467-2" H 0   0   50  0001 C CNN "mpn"
+F 6 "0" H 8550 4800 50  0001 C CNN "DNP"
 	1    8550 4800
 	1    0    0    -1
@@
 F 4 "Stackpole Electronics Inc" H 5250 3250 50  0001 C CNN "Manufacturer"
 F 5 "CF14JT1K00" H 5250 3250 50  0001 C CNN "mpn"
+F 6 "0" H 5250 3250 50  0001 C CNN "DNP"
 	1    5250 3250
 	0    1    1    0
@@
 F 4 "Stackpole Electronics Inc" H 5250 3400 50  0001 C CNN "Manufacturer"
 F 5 "CF14JT1K00" H 5250 3400 50  0001 C CNN "mpn"
+F 6 "0" H 5250 3400 50  0001 C CNN "DNP"
 	1    5250 3400
 	0    1    1    0
@@
 F 4 "Stackpole Electronics Inc" H 5250 3550 50  0001 C CNN "Manufacturer"
 F 5 "CF14JT1K00" H 5250 3550 50  0001 C CNN "mpn"
+F 6 "0" H 5250 3550 50  0001 C CNN "DNP"
 	1    5250 3550
 	0    1    1    0
@@
 F 4 "Vishay" H 0   0   50  0001 C CNN "Manufacturer"
 F 5 "K104K15X7RF5TL2" H 0   0   50  0001 C CNN "mpn"
+F 6 "0" H 2700 1850 50  0001 C CNN "DNP"
 	1    2700 1850
 	1    0    0    -1
@@
 F 4 "Vishay" H 0   0   50  0001 C CNN "Manufacturer"
 F 5 "K104K15X7RF5TL2" H 0   0   50  0001 C CNN "mpn"
+F 6 "0" H 2200 2800 50  0001 C CNN "DNP"
 	1    2200 2800
 	1    0    0    1
@@
 F 2 "Connector_PinHeader_2.54mm:PinHeader_2x03_P2.54mm_Vertical" V 6600 2300 50  0001 C CNN
 F 3 "~" H 5575 1700 50  0001 C CNN
-F 4 "~" H 6850 2250 50  0001 C CNN "Manufacturer"
-F 5 "~" H 6850 2250 50  0001 C CNN "mpn"
+F 4 "Harwin" H 6850 2250 50  0001 C CNN "Manufacturer"
+F 5 "M20-9760346" H 6850 2250 50  0001 C CNN "mpn"
+F 6 "0" H 6850 2250 50  0001 C CNN "DNP"
 	1    6850 2250
 	-1   0    0    -1
@@
 F 4 "Vishay" H 0   0   50  0001 C CNN "Manufacturer"
 F 5 "K104K15X7RF5TL2" H 0   0   50  0001 C CNN "mpn"
+F 6 "0" H 3400 1850 50  0001 C CNN "DNP"
 	1    3400 1850
 	1    0    0    -1
@@
 F 2 "Package_DIP:DIP-28_W7.62mm" H 3100 3800 50  0001 C CIN
 F 3 "http://ww1.microchip.com/downloads/en/DeviceDoc/ATmega328_P%20AVR%20MCU%20with%20picoPower%20Technology%20Data%20Sheet%2040001984A.pdf" H 3100 3800 50  0001 C CNN
-F 4 "Microchip" H 3100 3800 50  0001 C CNN "Manufacturer"
-F 5 "ATmega328-PU" H 3100 3800 50  0001 C CNN "mpn"
+F 4 "Microchip;On Shore Technology" H 3100 3800 50  0001 C CNN "Manufacturer"
+F 5 "ATmega328-PU;ED281DT" H 3100 3800 50  0001 C CNN "mpn"
+F 6 "0" H 3100 3800 50  0001 C CNN "DNP"
 	1    3100 3800
 	1    0    0    -1
@@
 F 4 "Kycon" H 9850 4000 50  0001 C CNN "Manufacturer"
 F 5 "KMDGX-6S-6S-S4N." H 9850 4000 50  0001 C CNN "mpn"
+F 6 "0" H 9850 4000 50  0001 C CNN "DNP"
 	1    9850 4000
 	1    0    0    -1
