File: neotron-32.sch (KiCad schematic (older format))
At the start: 12 parts, among them J1 Conn_02x06, J2 Conn_02x06, J3 Conn_02x04, U1 TM4C123G_Launchpad

Commit message: Adding MPNs.
Parts:
- R1, R2: Manufacturer (none) -> Stackpole Electronics Inc; PartNo (none) -> CF14JT1K00R
- RN1, RN2: Manufacturer (none) -> Bourns; PartNo (none) -> 4609X-101-473LF
- U1: Manufacturer (none) -> Texas Instruments; PartNo (none) -> EK-TM4C123GXL
Changed lines of the file:
@@
 F 2 "JGP Footprints:Launchpad_4x10" H 5700 2200 50  0001 C CNN
 F 3 "" H 5700 2200 50  0001 C CNN
+F 4 "Texas Instruments" H 5700 2200 50  0001 C CNN "Manufacturer"
+F 5 "EK-TM4C123GXL" H 5700 2200 50  0001 C CNN "PartNo"
 	1    5700 2200
 	1    0    0    -1
@@
 F 1 "47k x 8" V 1634 2250 50  0000 C CNN
 F 2 "Resistor_THT:R_Array_SIP9" V 1675 2250 50  0001 C CNN
-F 3 "http://www.vishay.com/docs/31509/csc.pdf" H 1200 2250 50  0001 C CNN
+F 3 "https://www.bourns.com/docs/Product-Datasheets/4600x.pdf" H 1200 2250 50  0001 C CNN
+F 4 "Bourns" H 1200 2250 50  0001 C CNN "Manufacturer"
+F 5 "4609X-101-473LF" H 1200 2250 50  0001 C CNN "PartNo"
 	1    1200 2250
 	0    -1   -1   0
@@
 F 1 "47k x 8" V 3184 2250 50  0000 C CNN
 F 2 "Resistor_THT:R_Array_SIP9" V 3225 2250 50  0001 C CNN
-F 3 "http://www.vishay.com/docs/31509/csc.pdf" H 2750 2250 50  0001 C CNN
+F 3 "https://www.bourns.com/docs/Product-Datasheets/4600x.pdf" H 2750 2250 50  0001 C CNN
+F 4 "Bourns" H 2750 2250 50  0001 C CNN "Manufacturer"
+F 5 "4609X-101-473LF" H 2750 2250 50  0001 C CNN "PartNo"
 	1    2750 2250
 	0    -1   -1   0
@@
 F 2 "Resistor_THT:R_Axial_DIN0207_L6.3mm_D2.5mm_P10.16mm_Horizontal" V 1230 1550 50  0001 C CNN
 F 3 "~" H 1300 1550 50  0001 C CNN
+F 4 "Stackpole Electronics Inc" H 1300 1550 50  0001 C CNN "Manufacturer"
+F 5 "CF14JT1K00R" H 1300 1550 50  0001 C CNN "PartNo"
 	1    1300 1550
 	0    1    1    0
@@
 F 2 "Resistor_THT:R_Axial_DIN0207_L6.3mm_D2.5mm_P10.16mm_Horizontal" V 1230 1350 50  0001 C CNN
 F 3 "~" H 1300 1350 50  0001 C CNN
+F 4 "Stackpole Electronics Inc" H 1300 1350 50  0001 C CNN "Manufacturer"
+F 5 "CF14JT1K00R" H 1300 1350 50  0001 C CNN "PartNo"
 	1    1300 1350
 	0    1    1    0

Commit message: Updated schematic on Windows.
Parts:
- U1: symbol TM4C_Launchpads:TM4C123G_Launchpad -> neotron-32-rescue:TM4C123G_Launchpad-TM4C_Launchpads
Changed lines of the file:
@@
 EESchema Schematic File Version 4
-EELAYER 30 0
+LIBS:neotron-32-cache
+EELAYER 26 0
 EELAYER END
 $Descr A4 11693 8268
@@
 	4900 2100 4150 2100
 $Comp
-L TM4C_Launchpads:TM4C123G_Launchpad U1
+L neotron-32-rescue:TM4C123G_Launchpad-TM4C_Launchpads U1
 U 1 1 5DF69932
 P 5700 2200

Commit message: Updated BOM.
Parts:
- J1, J2: Manufacturer (none) -> Harwin; PartNo (none) -> M20-9763646
- U1: Manufacturer Texas Instruments -> (none); PartNo EK-TM4C123GXL -> (none)
Changed lines of the file:
@@
 F 2 "Connector_PinHeader_2.54mm:PinHeader_2x06_P2.54mm_Vertical" H 8950 1050 50  0001 C CNN
 F 3 "~" H 8950 1050 50  0001 C CNN
+F 4 "Harwin" H 0   0   50  0001 C CNN "Manufacturer"
+F 5 "M20-9763646" H 0   0   50  0001 C CNN "PartNo"
 	1    8950 1050
 	1    0    0    -1
@@
 F 2 "Connector_PinHeader_2.54mm:PinHeader_2x06_P2.54mm_Vertical" H 8950 2050 50  0001 C CNN
 F 3 "~" H 8950 2050 50  0001 C CNN
+F 4 "Harwin" H 0   0   50  0001 C CNN "Manufacturer"
+F 5 "M20-9763646" H 0   0   50  0001 C CNN "PartNo"
 	1    8950 2050
 	1    0    0    -1
@@
 F 1 "TM4C123G_Launchpad" H 5700 3374 50  0000 C CNN
 F 2 "JGP Footprints:Launchpad_4x10" H 5700 2200 50  0001 C CNN
-F 3 "" H 5700 2200 50  0001 C CNN
-F 4 "Texas Instruments" H 5700 2200 50  0001 C CNN "Manufacturer"
-F 5 "EK-TM4C123GXL" H 5700 2200 50  0001 C CNN "PartNo"
+F 3 "~" H 5700 2200 50  0001 C CNN
+F 4 "~" H 5700 2200 50  0001 C CNN "Manufacturer"
+F 5 "~" H 5700 2200 50  0001 C CNN "PartNo"
 	1    5700 2200
 	1    0    0    -1
@@
 F 2 "Connector_PinHeader_2.54mm:PinHeader_2x04_P2.54mm_Vertical" H 8950 2950 50  0001 C CNN
 F 3 "~" H 8950 2950 50  0001 C CNN
+F 4 "~" H 0   0   50  0001 C CNN "Manufacturer"
+F 5 "~" H 0   0   50  0001 C CNN "PartNo"
 	1    8950 2950
 	1    0    0    -1
@@
 F 2 "MountingHole:MountingHole_3.2mm_M3" H 1550 6900 50  0001 C CNN
 F 3 "~" H 1550 6900 50  0001 C CNN
+F 4 "~" H 0   0   50  0001 C CNN "Manufacturer"
+F 5 "~" H 0   0   50  0001 C CNN "PartNo"
 	1    1550 6900
 	1    0    0    -1
@@
 F 2 "MountingHole:MountingHole_3.2mm_M3" H 1550 7100 50  0001 C CNN
 F 3 "~" H 1550 7100 50  0001 C CNN
+F 4 "~" H 0   0   50  0001 C CNN "Manufacturer"
+F 5 "~" H 0   0   50  0001 C CNN "PartNo"
 	1    1550 7100
 	1    0    0    -1
@@
 F 2 "MountingHole:MountingHole_3.2mm_M3" H 1550 7300 50  0001 C CNN
 F 3 "~" H 1550 7300 50  0001 C CNN
+F 4 "~" H 0   0   50  0001 C CNN "Manufacturer"
+F 5 "~" H 0   0   50  0001 C CNN "PartNo"
 	1    1550 7300
 	1    0    0    -1
@@
 F 2 "MountingHole:MountingHole_3.2mm_M3" H 1550 7500 50  0001 C CNN
 F 3 "~" H 1550 7500 50  0001 C CNN
+F 4 "~" H 0   0   50  0001 C CNN "Manufacturer"
+F 5 "~" H 0   0   50  0001 C CNN "PartNo"
 	1    1550 7500
 	1    0    0    -1

Commit message: Add some extra explanatory notes.
Other:
- note added: "The Neotron-32 is based around a Texas Instruments EK-TM4C123GH6 Tiva-C Launchpad board. This includes a TM4C123 microcontroller\nand a JTAG + USB Serial interface.\n\nDrill down into the sub-sheets to see more detail."
- moved on the sheet: H1, H2, H3, H4
Changed lines of the file:
@@
 EESchema Schematic File Version 4
-LIBS:neotron-32-cache
-EELAYER 26 0
+EELAYER 30 0
 EELAYER END
 $Descr A4 11693 8268
@@
 L Mechanical:MountingHole H1
 U 1 1 5DFC719B
-P 1550 6900
-F 0 "H1" H 1650 6946 50  0000 L CNN
-F 1 "MountingHole" H 1650 6855 50  0000 L CNN
-F 2 "MountingHole:MountingHole_3.2mm_M3" H 1550 6900 50  0001 C CNN
-F 3 "~" H 1550 6900 50  0001 C CNN
-F 4 "~" H 0   0   50  0001 C CNN "Manufacturer"
-F 5 "~" H 0   0   50  0001 C CNN "PartNo"
-	1    1550 6900
+P 6200 6800
+F 0 "H1" H 6300 6846 50  0000 L CNN
+F 1 "MountingHole" H 6300 6755 50  0000 L CNN
+F 2 "MountingHole:MountingHole_3.2mm_M3" H 6200 6800 50  0001 C CNN
+F 3 "~" H 6200 6800 50  0001 C CNN
+F 4 "~" H 4650 -100 50  0001 C CNN "Manufacturer"
+F 5 "~" H 4650 -100 50  0001 C CNN "PartNo"
+	1    6200 6800
 	1    0    0    -1
 $EndComp
@@
 L Mechanical:MountingHole H2
 U 1 1 5DFC7744
-P 1550 7100
-F 0 "H2" H 1650 7146 50  0000 L CNN
-F 1 "MountingHole" H 1650 7055 50  0000 L CNN
-F 2 "MountingHole:MountingHole_3.2mm_M3" H 1550 7100 50  0001 C CNN
-F 3 "~" H 1550 7100 50  0001 C CNN
-F 4 "~" H 0   0   50  0001 C CNN "Manufacturer"
-F 5 "~" H 0   0   50  0001 C CNN "PartNo"
-	1    1550 7100
+P 6200 7000
+F 0 "H2" H 6300 7046 50  0000 L CNN
+F 1 "MountingHole" H 6300 6955 50  0000 L CNN
+F 2 "MountingHole:MountingHole_3.2mm_M3" H 6200 7000 50  0001 C CNN
+F 3 "~" H 6200 7000 50  0001 C CNN
+F 4 "~" H 4650 -100 50  0001 C CNN "Manufacturer"
+F 5 "~" H 4650 -100 50  0001 C CNN "PartNo"
+	1    6200 7000
 	1    0    0    -1
 $EndComp
@@
 L Mechanical:MountingHole H3
 U 1 1 5DFC781B
-P 1550 7300
-F 0 "H3" H 1650 7346 50  0000 L CNN
-F 1 "MountingHole" H 1650 7255 50  0000 L CNN
-F 2 "MountingHole:MountingHole_3.2mm_M3" H 1550 7300 50  0001 C CNN
-F 3 "~" H 1550 7300 50  0001 C CNN
-F 4 "~" H 0   0   50  0001 C CNN "Manufacturer"
-F 5 "~" H 0   0   50  0001 C CNN "PartNo"
-	1    1550 7300
+P 6200 7200
+F 0 "H3" H 6300 7246 50  0000 L CNN
+F 1 "MountingHole" H 6300 7155 50  0000 L CNN
+F 2 "MountingHole:MountingHole_3.2mm_M3" H 6200 7200 50  0001 C CNN
+F 3 "~" H 6200 7200 50  0001 C CNN
+F 4 "~" H 4650 -100 50  0001 C CNN "Manufacturer"
+F 5 "~" H 4650 -100 50  0001 C CNN "PartNo"
+	1    6200 7200
 	1    0    0    -1
 $EndComp
@@
 L Mechanical:MountingHole H4
 U 1 1 5DFC799C
-P 1550 7500
-F 0 "H4" H 1650 7546 50  0000 L CNN
-F 1 "MountingHole" H 1650 7455 50  0000 L CNN
-F 2 "MountingHole:MountingHole_3.2mm_M3" H 1550 7500 50  0001 C CNN
-F 3 "~" H 1550 7500 50  0001 C CNN
-F 4 "~" H 0   0   50  0001 C CNN "Manufacturer"
-F 5 "~" H 0   0   50  0001 C CNN "PartNo"
-	1    1550 7500
+P 6200 7400
+F 0 "H4" H 6300 7446 50  0000 L CNN
+F 1 "MountingHole" H 6300 7355 50  0000 L CNN
+F 2 "MountingHole:MountingHole_3.2mm_M3" H 6200 7400 50  0001 C CNN
+F 3 "~" H 6200 7400 50  0001 C CNN
+F 4 "~" H 4650 -100 50  0001 C CNN "Manufacturer"
+F 5 "~" H 4650 -100 50  0001 C CNN "PartNo"
+	1    6200 7400
 	1    0    0    -1
 $EndComp
@@
 Wire Wire Line
 	8250 1550 9950 1550
+Text Notes 550  7700 0    50   Italic 0
+The Neotron-32 is based around a Texas Instruments EK-TM4C123GH6 Tiva-C Launchpad board. This includes a TM4C123 microcontroller\nand a JTAG + USB Serial interface.\n\nDrill down into the sub-sheets to see more detail.
 Wire Bus Line
 	8150 2900 8150 3450

Commit message: Fix Stackpole 1K part number.
Parts:
- R1, R2: PartNo CF14JT1K00R -> CF14JT1K00
Changed lines of the file:
@@
 F 3 "~" H 1300 1550 50  0001 C CNN
 F 4 "Stackpole Electronics Inc" H 1300 1550 50  0001 C CNN "Manufacturer"
-F 5 "CF14JT1K00R" H 1300 1550 50  0001 C CNN "PartNo"
+F 5 "CF14JT1K00" H 1300 1550 50  0001 C CNN "PartNo"
 	1    1300 1550
 	0    1    1    0
@@
 F 3 "~" H 1300 1350 50  0001 C CNN
 F 4 "Stackpole Electronics Inc" H 1300 1350 50  0001 C CNN "Manufacturer"
-F 5 "CF14JT1K00R" H 1300 1350 50  0001 C CNN "PartNo"
+F 5 "CF14JT1K00" H 1300 1350 50  0001 C CNN "PartNo"
 	1    1300 1350
 	0    1    1    0
