File: power.sch (KiCad schematic (older format))
At the start: 11 parts, among them J9 USB_B, SW1 SW_SPST, SW2 SW_Push, U4 TC1262-33

Commit message: Adding MPNs.
Parts:
- D2: Manufacturer (none) -> Littelfuse; PartNo (none) -> SA5.0A
- R28: Manufacturer (none) -> Stackpole Electronics Inc; PartNo (none) -> CF14JT330R
- SW1, SW2: Manufacturer (none) -> Harwin; PartNo (none) -> M20-9990246
- U4: Manufacturer (none) -> Microchip; PartNo (none) -> TC1262-3.3VAB
Changed lines of the file:
@@
 F 3 "https://www.littelfuse.com/~/media/electronics/datasheets/tvs_diodes/littelfuse_tvs_diode_sa_datasheet.pdf.pdf" H 5050 3600 50  0001 C CNN
 F 4 "SA5.0ALFCT-ND " V 5050 3600 50  0001 C CNN "Digikey"
+F 5 "Littelfuse" H 5050 3600 50  0001 C CNN "Manufacturer"
+F 6 "SA5.0A" H 5050 3600 50  0001 C CNN "PartNo"
 	1    5050 3600
 	0    1    1    0
@@
 F 2 "Connector_PinHeader_2.54mm:PinHeader_1x02_P2.54mm_Vertical" H 8150 3900 50  0001 C CNN
 F 3 "~" H 8150 3900 50  0001 C CNN
+F 4 "Harwin" H 8150 3700 50  0001 C CNN "Manufacturer"
+F 5 "M20-9990246" H 8150 3700 50  0001 C CNN "PartNo"
 	1    8150 3700
 	1    0    0    -1
@@
 F 2 "Package_TO_SOT_THT:TO-220-3_Vertical" H 6900 3525 50  0001 C CIN
 F 3 "http://ww1.microchip.com/downloads/en/DeviceDoc/21373C.pdf" H 6900 3000 50  0001 C CNN
+F 4 "Microchip" H 6900 3300 50  0001 C CNN "Manufacturer"
+F 5 "TC1262-3.3VAB" H 6900 3300 50  0001 C CNN "PartNo"
 	1    6900 3300
 	1    0    0    -1
@@
 F 2 "Connector_PinHeader_2.54mm:PinHeader_1x02_P2.54mm_Vertical" H 3850 3300 50  0001 C CNN
 F 3 "~" H 3850 3300 50  0001 C CNN
+F 4 "Harwin" H 3850 3300 50  0001 C CNN "Manufacturer"
+F 5 "M20-9990246" H 3850 3300 50  0001 C CNN "PartNo"
 	1    3850 3300
 	1    0    0    -1
@@
 F 2 "Resistor_THT:R_Axial_DIN0207_L6.3mm_D2.5mm_P10.16mm_Horizontal" V 8530 3700 50  0001 C CNN
 F 3 "~" H 8600 3700 50  0001 C CNN
+F 4 "Stackpole Electronics Inc" H 8600 3700 50  0001 C CNN "Manufacturer"
+F 5 "CF14JT330R" H 8600 3700 50  0001 C CNN "PartNo"
 	1    8600 3700
 	0    1    1    0

Commit message: Updated BOM.
Parts:
- C6: Manufacturer (none) -> Vishay; PartNo (none) -> MAL203858109E3
- C7: Manufacturer (none) -> Vishay; PartNo (none) -> K104K15X7RF5TL2
- C8: Manufacturer (none) -> Vishay; PartNo (none) -> MAL214250479E3
- D2: Digikey SA5.0ALFCT-ND -> (none)
- F1: Digikey RXEF025HF-ND -> (none)
- J9: Manufacturer (none) -> On Shore Technology; PartNo (none) -> USB-B1HSB6; RS (none) -> USB-B1HSB6
Changed lines of the file:
@@
 F 1 "USB_B" H 3050 3850 50  0000 C CNN
 F 2 "Connector_USB:USB_B_OST_USB-B1HSxx_Horizontal" H 3200 3450 50  0001 C CNN
-F 3 " ~" H 3200 3450 50  0001 C CNN
+F 3 "http://www.on-shore.com/wp-content/uploads/USB-B1HSXX.pdf" H 3200 3450 50  0001 C CNN
+F 4 "On Shore Technology" H 0   0   50  0001 C CNN "Manufacturer"
+F 5 "USB-B1HSB6" H 0   0   50  0001 C CNN "PartNo"
+F 6 "USB-B1HSB6 " H 0   0   50  0001 C CNN "RS"
 	1    3050 3500
 	1    0    0    -1
@@
 F 2 "Capacitor_THT:CP_Radial_D6.3mm_P2.50mm" H 5588 3450 50  0001 C CNN
 F 3 "~" H 5550 3600 50  0001 C CNN
+F 4 "Vishay" H 0   0   50  0001 C CNN "Manufacturer"
+F 5 "MAL203858109E3" H 0   0   50  0001 C CNN "PartNo"
 	1    5550 3600
 	1    0    0    -1
@@
 F 2 "Capacitor_THT:C_Disc_D3.0mm_W2.0mm_P2.50mm" H 5988 3450 50  0001 C CNN
 F 3 "~" H 5950 3600 50  0001 C CNN
+F 4 "Vishay" H 0   0   50  0001 C CNN "Manufacturer"
+F 5 "K104K15X7RF5TL2" H 0   0   50  0001 C CNN "PartNo"
 	1    5950 3600
 	1    0    0    -1
@@
 F 2 "Diode_THT:D_DO-15_P10.16mm_Horizontal" H 4750 3100 50  0001 L CNN
 F 3 "https://www.littelfuse.com/~/media/electronics/product_specifications/resettable_ptcs/littelfuse_ptc_rxef025_product_specification.pdf.pdf" H 4700 3300 50  0001 C CNN
-F 4 "RXEF025HF-ND" V 4700 3300 50  0001 C CNN "Digikey"
+F 4 "" V 4700 3300 50  0001 C CNN "Digikey"
 F 5 "Littelfuse Inc" V 4700 3300 50  0001 C CNN "Manufacturer"
 F 6 "RXEF025" V 4700 3300 50  0001 C CNN "PartNo"
@@
 F 2 "Diode_THT:D_DO-15_P12.70mm_Horizontal" H 5050 3600 50  0001 C CNN
 F 3 "https://www.littelfuse.com/~/media/electronics/datasheets/tvs_diodes/littelfuse_tvs_diode_sa_datasheet.pdf.pdf" H 5050 3600 50  0001 C CNN
-F 4 "SA5.0ALFCT-ND " V 5050 3600 50  0001 C CNN "Digikey"
+F 4 "" V 5050 3600 50  0001 C CNN "Digikey"
 F 5 "Littelfuse" H 5050 3600 50  0001 C CNN "Manufacturer"
 F 6 "SA5.0A" H 5050 3600 50  0001 C CNN "PartNo"
@@
 F 2 "Resistor_THT:R_Axial_DIN0207_L6.3mm_D2.5mm_P10.16mm_Horizontal" V 2880 4100 50  0001 C CNN
 F 3 "~" H 2950 4100 50  0001 C CNN
+F 4 "~" H 0   0   50  0001 C CNN "Manufacturer"
+F 5 "~" H 0   0   50  0001 C CNN "PartNo"
 	1    2950 4100
 	-1   0    0    1
@@
 F 2 "Capacitor_THT:CP_Radial_D6.3mm_P2.50mm" H 7388 3450 50  0001 C CNN
 F 3 "~" H 7350 3600 50  0001 C CNN
+F 4 "Vishay" H 0   0   50  0001 C CNN "Manufacturer"
+F 5 "MAL214250479E3" H 0   0   50  0001 C CNN "PartNo"
 	1    7350 3600
 	1    0    0    -1

Commit message: Removed Digikey and RS part numbers.
Parts:
- J9: RS USB-B1HSB6 -> (none)
Changed lines of the file:
@@
 F 4 "On Shore Technology" H 0   0   50  0001 C CNN "Manufacturer"
 F 5 "USB-B1HSB6" H 0   0   50  0001 C CNN "PartNo"
-F 6 "USB-B1HSB6 " H 0   0   50  0001 C CNN "RS"
 	1    3050 3500
 	1    0    0    -1
@@
 F 2 "Diode_THT:D_DO-15_P10.16mm_Horizontal" H 4750 3100 50  0001 L CNN
 F 3 "https://www.littelfuse.com/~/media/electronics/product_specifications/resettable_ptcs/littelfuse_ptc_rxef025_product_specification.pdf.pdf" H 4700 3300 50  0001 C CNN
-F 4 "" V 4700 3300 50  0001 C CNN "Digikey"
 F 5 "Littelfuse Inc" V 4700 3300 50  0001 C CNN "Manufacturer"
 F 6 "RXEF025" V 4700 3300 50  0001 C CNN "PartNo"
@@
 F 2 "Diode_THT:D_DO-15_P12.70mm_Horizontal" H 5050 3600 50  0001 C CNN
 F 3 "https://www.littelfuse.com/~/media/electronics/datasheets/tvs_diodes/littelfuse_tvs_diode_sa_datasheet.pdf.pdf" H 5050 3600 50  0001 C CNN
-F 4 "" V 5050 3600 50  0001 C CNN "Digikey"
 F 5 "Littelfuse" H 5050 3600 50  0001 C CNN "Manufacturer"
 F 6 "SA5.0A" H 5050 3600 50  0001 C CNN "PartNo"

Commit message: Add some extra explanatory notes.
Other:
- note added: "Connect to a 5V USB Power Supply. The board should only use around 100 mA in operation, so almost any USB 'phone charger'\nshould work, provided you have a full-size USB B cable (rather than USB micro-B). We use the full-size B as it is easier to solder the\nconnector.\n\nWe have our own 3.3V LDO to avoid overloading the LDO on the Launchpad.\n\nTaking the RESET pin low should reset the Launchpad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"
Changed lines of the file:
@@
 EESchema Schematic File Version 4
-LIBS:neotron-32-cache
-EELAYER 26 0
+EELAYER 30 0
 EELAYER END
 $Descr A4 11693 8268
@@
 F 2 "Diode_THT:D_DO-15_P10.16mm_Horizontal" H 4750 3100 50  0001 L CNN
 F 3 "https://www.littelfuse.com/~/media/electronics/product_specifications/resettable_ptcs/littelfuse_ptc_rxef025_product_specification.pdf.pdf" H 4700 3300 50  0001 C CNN
-F 5 "Littelfuse Inc" V 4700 3300 50  0001 C CNN "Manufacturer"
-F 6 "RXEF025" V 4700 3300 50  0001 C CNN "PartNo"
+F 4 "Littelfuse Inc" V 4700 3300 50  0001 C CNN "Manufacturer"
+F 5 "RXEF025" V 4700 3300 50  0001 C CNN "PartNo"
 	1    4700 3300
 	0    1    1    0
@@
 F 2 "Diode_THT:D_DO-15_P12.70mm_Horizontal" H 5050 3600 50  0001 C CNN
 F 3 "https://www.littelfuse.com/~/media/electronics/datasheets/tvs_diodes/littelfuse_tvs_diode_sa_datasheet.pdf.pdf" H 5050 3600 50  0001 C CNN
-F 5 "Littelfuse" H 5050 3600 50  0001 C CNN "Manufacturer"
-F 6 "SA5.0A" H 5050 3600 50  0001 C CNN "PartNo"
+F 4 "Littelfuse" H 5050 3600 50  0001 C CNN "Manufacturer"
+F 5 "SA5.0A" H 5050 3600 50  0001 C CNN "PartNo"
 	1    5050 3600
 	0    1    1    0
@@
 Text Notes 8000 3950 0    50   ~ 0
 330R is for current limiting
+Text Notes 550  7700 0    50   Italic 0
+Connect to a 5V USB Power Supply. The board should only use around 100 mA in operation, so almost any USB 'phone charger'\nshould work, provided you have a full-size USB B cable (rather than USB micro-B). We use the full-size B as it is easier to solder the\nconnector.\n\nWe have our own 3.3V LDO to avoid overloading the LDO on the Launchpad.\n\nTaking the RESET pin low should reset the Launchpad, the AtMega and the MCP23S17.
 $EndSCHEMATC
