File: storage.sch (KiCad schematic (older format))
At the start: 8 parts, among them J10 Amphenol micro SD 114-00841-68, U2 74LS14

Commit message: Adding MPNs.
Parts:
- R15, R16: Manufacturer (none) -> Stackpole Electronics Inc; PartNo (none) -> CF14JT47K0
- R17: Manufacturer (none) -> Stackpole Electronics Inc; PartNo (none) -> CF14JT330R
- U2: Manufacturer (none) -> Texas Instruments; PartNo (none) -> SN74LS14N
Changed lines of the file:
@@
 F 2 "Resistor_THT:R_Axial_DIN0207_L6.3mm_D2.5mm_P10.16mm_Horizontal" V 4480 2900 50  0001 C CNN
 F 3 "~" H 4550 2900 50  0001 C CNN
+F 4 "Stackpole Electronics Inc" H 4550 2900 50  0001 C CNN "Manufacturer"
+F 5 "CF14JT47K0" H 4550 2900 50  0001 C CNN "PartNo"
 	1    4550 2900
 	0    1    1    0
@@
 F 2 "Resistor_THT:R_Axial_DIN0207_L6.3mm_D2.5mm_P10.16mm_Horizontal" V 4480 2700 50  0001 C CNN
 F 3 "~" H 4550 2700 50  0001 C CNN
+F 4 "Stackpole Electronics Inc" H 4550 2700 50  0001 C CNN "Manufacturer"
+F 5 "CF14JT47K0" H 4550 2700 50  0001 C CNN "PartNo"
 	1    4550 2700
 	0    1    1    0
@@
 F 2 "Resistor_THT:R_Axial_DIN0207_L6.3mm_D2.5mm_P10.16mm_Horizontal" V 7080 2050 50  0001 C CNN
 F 3 "~" H 7150 2050 50  0001 C CNN
+F 4 "Stackpole Electronics Inc" H 7150 2050 50  0001 C CNN "Manufacturer"
+F 5 "CF14JT330R" H 7150 2050 50  0001 C CNN "PartNo"
 	1    7150 2050
 	0    1    1    0
@@
 F 2 "Package_DIP:DIP-14_W7.62mm" H 5850 2050 50  0001 C CNN
 F 3 "http://www.ti.com/lit/gpn/sn74LS14" H 5850 2050 50  0001 C CNN
+F 4 "Texas Instruments" H 5850 2050 50  0001 C CNN "Manufacturer"
+F 5 "SN74LS14N" H 5850 2050 50  0001 C CNN "PartNo"
 	6    5850 2050
 	1    0    0    -1
@@
 F 2 "Package_DIP:DIP-14_W7.62mm" H 6550 2050 50  0001 C CNN
 F 3 "http://www.ti.com/lit/gpn/sn74LS14" H 6550 2050 50  0001 C CNN
+F 4 "Texas Instruments" H 6550 2050 50  0001 C CNN "Manufacturer"
+F 5 "SN74LS14N" H 6550 2050 50  0001 C CNN "PartNo"
 	5    6550 2050
 	1    0    0    -1

Commit message: Updated schematic on Windows.
Parts:
- J10: symbol Connector:Micro_SD_Card -> neotron-32-rescue:Micro_SD_Card-Connector
Changed lines of the file:
@@
 EESchema Schematic File Version 4
-EELAYER 30 0
+LIBS:neotron-32-cache
+EELAYER 26 0
 EELAYER END
 $Descr A4 11693 8268
@@
 	7300 4000 7300 4100
 $Comp
-L Connector:Micro_SD_Card J10
+L neotron-32-rescue:Micro_SD_Card-Connector J10
 U 1 1 5E19DB95
 P 6250 3400
+AR Path="/5E19DB95" Ref="J10"  Part="1"
+AR Path="/5DF1D0B0/5E19DB95" Ref="J10"  Part="1"
 F 0 "J10" H 6200 4117 50  0000 C CNN
 F 1 "Amphenol micro SD 114-00841-68" H 6200 4026 50  0000 C CNN

Commit message: Updated BOM.
Parts:
- C9: Manufacturer (none) -> Vishay; PartNo (none) -> K104K15X7RF5TL2
- D3: Manufacturer (none) -> Würth Elektronik; PartNo (none) -> 151031SS04000
- J10: Manufacturer (none) -> Amphenol; PartNo (none) -> 114-00841-68
Changed lines of the file:
@@
 F 2 "Resistor_THT:R_Axial_DIN0207_L6.3mm_D2.5mm_P10.16mm_Horizontal" V 7230 4250 50  0001 C CNN
 F 3 "~" H 7300 4250 50  0001 C CNN
+F 4 "~" H 0   0   50  0001 C CNN "Manufacturer"
+F 5 "~" H 0   0   50  0001 C CNN "PartNo"
 	1    7300 4250
 	1    0    0    -1
@@
 F 2 "Capacitor_THT:C_Disc_D3.0mm_W2.0mm_P2.50mm" H 7938 3350 50  0001 C CNN
 F 3 "~" H 7900 3500 50  0001 C CNN
+F 4 "Vishay" H 0   0   50  0001 C CNN "Manufacturer"
+F 5 "K104K15X7RF5TL2" H 0   0   50  0001 C CNN "PartNo"
 	1    7900 3500
 	1    0    0    -1
@@
 F 2 "LED_THT:LED_D3.0mm" H 7600 2050 50  0001 C CNN
 F 3 "~" H 7600 2050 50  0001 C CNN
+F 4 "Würth Elektronik" H 0   0   50  0001 C CNN "Manufacturer"
+F 5 "151031SS04000" H 0   0   50  0001 C CNN "PartNo"
 	1    7600 2050
 	1    0    0    -1
@@
 F 2 "Amphenol SD Card:1140084168" H 7400 3700 50  0001 C CNN
 F 3 "https://media.digikey.com/pdf/Data%20Sheets/Amphenol%20PDFs/114-00841-68.pdf" H 6250 3400 50  0001 C CNN
+F 4 "Amphenol" H 0   0   50  0001 C CNN "Manufacturer"
+F 5 "114-00841-68" H 0   0   50  0001 C CNN "PartNo"
 	1    6250 3400
 	1    0    0    -1

Commit message: Add some extra explanatory notes.
Other:
- note added: "We use a micro-SD card for space reasons. The SD card is driven in SPI mode."
- note removed: "SD Card Storage"
Changed lines of the file:
@@
 EESchema Schematic File Version 4
-LIBS:neotron-32-cache
-EELAYER 26 0
+EELAYER 30 0
 EELAYER END
 $Descr A4 11693 8268
@@
 Wire Wire Line
 	4050 2900 4050 3400
-Text Notes 5400 1500 0    100  ~ 20
-SD Card Storage
+Text Notes 550  7700 0    50   Italic 0
+We use a micro-SD card for space reasons. The SD card is driven in SPI mode.
 $EndSCHEMATC
