File: storage.sch (KiCad schematic (older format))
At the start: 8 parts, among them J10 Amphenol micro SD 114-00841-68, U2 74LS14

Commit message: Replace Amphenol SD connector with Molex.
The Molex connector has the pins at the rear, which means you can blob
down solder without fouling the card insertion.
Parts:
- J10: value Amphenol micro SD 114-00841-68 -> micro SD Card; footprint Amphenol SD Card:1140084168 -> JGP Footprints:Molex_4730_2651; symbol neotron-32-rescue:Micro_SD_Card-Connector -> Connector:Micro_SD_Card; Manufacturer Amphenol -> Molex; PartNo 114-00841-68 -> 47309-2651
Changed lines of the file:
@@
 	7300 4000 7300 4100
 $Comp
-L neotron-32-rescue:Micro_SD_Card-Connector J10
+L Connector:Micro_SD_Card J10
 U 1 1 5E19DB95
 P 6250 3400
@@
 AR Path="/5DF1D0B0/5E19DB95" Ref="J10"  Part="1"
 F 0 "J10" H 6200 4117 50  0000 C CNN
-F 1 "Amphenol micro SD 114-00841-68" H 6200 4026 50  0000 C CNN
-F 2 "Amphenol SD Card:1140084168" H 7400 3700 50  0001 C CNN
-F 3 "https://media.digikey.com/pdf/Data%20Sheets/Amphenol%20PDFs/114-00841-68.pdf" H 6250 3400 50  0001 C CNN
-F 4 "Amphenol" H 0   0   50  0001 C CNN "Manufacturer"
-F 5 "114-00841-68" H 0   0   50  0001 C CNN "PartNo"
+F 1 "micro SD Card" H 6200 4026 50  0000 C CNN
+F 2 "JGP Footprints:Molex_4730_2651" H 7400 3700 50  0001 C CNN
+F 3 "" H 6250 3400 50  0001 C CNN
+F 4 "Molex" H 0   0   50  0001 C CNN "Manufacturer"
+F 5 "47309-2651" H 0   0   50  0001 C CNN "PartNo"
 	1    6250 3400
 	1    0    0    -1

Commit message: Moved non-standard components into local libraries.
neotron-32.lib is the symbol library.
neotron-32.pretty is the footprint library.

Also swapped the DE9 and DB25 headers for IDC boxed versions. Involved
moving a resistor out of the way.

The Keystone 103 battery holder is a straight copy of the standard
footprint, but with the Courtyard removed to bypass the 'Courtyard is
not closed' DRC error.
Parts:
- J10: footprint JGP Footprints:Molex_4730_2651 -> Neotron 32:Molex_4730_2651
Changed lines of the file:
@@
 F 0 "J10" H 6200 4117 50  0000 C CNN
 F 1 "micro SD Card" H 6200 4026 50  0000 C CNN
-F 2 "JGP Footprints:Molex_4730_2651" H 7400 3700 50  0001 C CNN
+F 2 "Neotron 32:Molex_4730_2651" H 7400 3700 50  0001 C CNN
 F 3 "" H 6250 3400 50  0001 C CNN
 F 4 "Molex" H 0   0   50  0001 C CNN "Manufacturer"
