File: midi.sch (KiCad schematic (older format))
At the start: 14 parts, among them J4 DIN-5 MIDI Through, J5 DIN-5 MIDI In, J6 DIN-5 MIDI Out, U2 74LS14, U3 6N138

Commit message: Adding MPNs.
Parts:
- R3, R4, R5, R6, R7: Manufacturer (none) -> Stackpole Electronics Inc; PartNo (none) -> CF14JT220R
- R8: Manufacturer (none) -> Stackpole Electronics Inc; PartNo (none) -> CF14JT10K0
- R9: Manufacturer (none) -> Stackpole Electronics Inc; PartNo (none) -> CF14JT470R
- U2: Manufacturer (none) -> Texas Instruments; PartNo (none) -> SN74LS14N
- U3: Manufacturer (none) -> Lite-On Inc.; PartNo (none) -> 6N138
Changed lines of the file:
@@
 F 1 "6N138" H 4900 4026 50  0000 C CNN
 F 2 "Package_DIP:DIP-8_W7.62mm" H 5190 3350 50  0001 C CNN
-F 3 "http://www.onsemi.com/pub/Collateral/HCPL2731-D.pdf" H 5190 3350 50  0001 C CNN
+F 3 "https://media.digikey.com/pdf/Data%20Sheets/Lite-On%20PDFs/6N138-39%20Series.pdf" H 5190 3350 50  0001 C CNN
+F 4 "Lite-On Inc." H 4900 3650 50  0001 C CNN "Manufacturer"
+F 5 "6N138" H 4900 3650 50  0001 C CNN "PartNo"
 	1    4900 3650
 	1    0    0    -1
@@
 F 2 "Package_DIP:DIP-14_W7.62mm" H 3900 2650 50  0001 C CNN
 F 3 "http://www.ti.com/lit/gpn/sn74LS14" H 3900 2650 50  0001 C CNN
+F 4 "Texas Instruments" H 3900 2650 50  0001 C CNN "Manufacturer"
+F 5 "SN74LS14N" H 3900 2650 50  0001 C CNN "PartNo"
 	1    3900 2650
 	-1   0    0    1
@@
 F 2 "Package_DIP:DIP-14_W7.62mm" H 4800 2650 50  0001 C CNN
 F 3 "http://www.ti.com/lit/gpn/sn74LS14" H 4800 2650 50  0001 C CNN
+F 4 "Texas Instruments" H 4800 2650 50  0001 C CNN "Manufacturer"
+F 5 "SN74LS14N" H 4800 2650 50  0001 C CNN "PartNo"
 	2    4800 2650
 	-1   0    0    1
@@
 F 2 "Package_DIP:DIP-14_W7.62mm" H 4800 4750 50  0001 C CNN
 F 3 "http://www.ti.com/lit/gpn/sn74LS14" H 4800 4750 50  0001 C CNN
+F 4 "Texas Instruments" H 4800 4750 50  0001 C CNN "Manufacturer"
+F 5 "SN74LS14N" H 4800 4750 50  0001 C CNN "PartNo"
 	3    4800 4750
 	-1   0    0    1
@@
 F 2 "Package_DIP:DIP-14_W7.62mm" H 3900 4750 50  0001 C CNN
 F 3 "http://www.ti.com/lit/gpn/sn74LS14" H 3900 4750 50  0001 C CNN
+F 4 "Texas Instruments" H 3900 4750 50  0001 C CNN "Manufacturer"
+F 5 "SN74LS14N" H 3900 4750 50  0001 C CNN "PartNo"
 	4    3900 4750
 	-1   0    0    1
@@
 F 2 "Package_DIP:DIP-14_W7.62mm" H 8000 3600 50  0001 C CNN
 F 3 "http://www.ti.com/lit/gpn/sn74LS14" H 8000 3600 50  0001 C CNN
+F 4 "Texas Instruments" H 8000 3600 50  0001 C CNN "Manufacturer"
+F 5 "SN74LS14N" H 8000 3600 50  0001 C CNN "PartNo"
 	7    8000 3600
 	1    0    0    -1
@@
 F 2 "Resistor_THT:R_Axial_DIN0207_L6.3mm_D2.5mm_P10.16mm_Horizontal" V 3130 3300 50  0001 C CNN
 F 3 "~" H 3200 3300 50  0001 C CNN
+F 4 "Stackpole Electronics Inc" H 3200 3300 50  0001 C CNN "Manufacturer"
+F 5 "CF14JT220R" H 3200 3300 50  0001 C CNN "PartNo"
 	1    3200 3300
 	0    1    1    0
@@
 F 2 "Resistor_THT:R_Axial_DIN0207_L6.3mm_D2.5mm_P10.16mm_Horizontal" V 3230 2650 50  0001 C CNN
 F 3 "~" H 3300 2650 50  0001 C CNN
+F 4 "Stackpole Electronics Inc" H 3300 2650 50  0001 C CNN "Manufacturer"
+F 5 "CF14JT220R" H 3300 2650 50  0001 C CNN "PartNo"
 	1    3300 2650
 	0    1    1    0
@@
 F 2 "Resistor_THT:R_Axial_DIN0207_L6.3mm_D2.5mm_P10.16mm_Horizontal" V 3230 4750 50  0001 C CNN
 F 3 "~" H 3300 4750 50  0001 C CNN
+F 4 "Stackpole Electronics Inc" H 3300 4750 50  0001 C CNN "Manufacturer"
+F 5 "CF14JT220R" H 3300 4750 50  0001 C CNN "PartNo"
 	1    3300 4750
 	0    1    1    0
@@
 F 2 "Resistor_THT:R_Axial_DIN0207_L6.3mm_D2.5mm_P10.16mm_Horizontal" V 5480 3350 50  0001 C CNN
 F 3 "~" H 5550 3350 50  0001 C CNN
+F 4 "Stackpole Electronics Inc" H 5550 3350 50  0001 C CNN "Manufacturer"
+F 5 "CF14JT470R" H 5550 3350 50  0001 C CNN "PartNo"
 	1    5550 3350
 	-1   0    0    1
@@
 F 2 "Resistor_THT:R_Axial_DIN0207_L6.3mm_D2.5mm_P10.16mm_Horizontal" V 5330 4000 50  0001 C CNN
 F 3 "~" H 5400 4000 50  0001 C CNN
+F 4 "Stackpole Electronics Inc" H 5400 4000 50  0001 C CNN "Manufacturer"
+F 5 "CF14JT10K0" H 5400 4000 50  0001 C CNN "PartNo"
 	1    5400 4000
 	-1   0    0    1
@@
 F 2 "Resistor_THT:R_Axial_DIN0207_L6.3mm_D2.5mm_P10.16mm_Horizontal" V 1980 4450 50  0001 C CNN
 F 3 "~" H 2050 4450 50  0001 C CNN
+F 4 "Stackpole Electronics Inc" H 2050 4450 50  0001 C CNN "Manufacturer"
+F 5 "CF14JT220R" H 2050 4450 50  0001 C CNN "PartNo"
 	1    2050 4450
 	-1   0    0    1
@@
 F 2 "Resistor_THT:R_Axial_DIN0207_L6.3mm_D2.5mm_P10.16mm_Horizontal" V 1980 2350 50  0001 C CNN
 F 3 "~" H 2050 2350 50  0001 C CNN
+F 4 "Stackpole Electronics Inc" H 2050 2350 50  0001 C CNN "Manufacturer"
+F 5 "CF14JT220R" H 2050 2350 50  0001 C CNN "PartNo"
 	1    2050 2350
 	-1   0    0    1

Commit message: Fix MIDI Out/Through mix-up.
Parts:
- J4: value DIN-5 MIDI Through -> DIN-5 MIDI Out
- J6: value DIN-5 MIDI Out -> DIN-5 MIDI Through
Changed lines of the file:
@@
 AR Path="/5DF253FB/5DF53872" Ref="J4"  Part="1"
 F 0 "J4" H 2600 2425 50  0000 C CNN
-F 1 "DIN-5 MIDI Through" H 2600 2334 50  0000 C CNN
+F 1 "DIN-5 MIDI Out" H 2600 2334 50  0000 C CNN
 F 2 "JGP Footprints:5P180 DIN Socket" H 2600 2700 50  0001 C CNN
 F 3 "http://www.mouser.com/ds/2/18/40_c091_abd_e-75918.pdf" H 2600 2700 50  0001 C CNN
@@
 AR Path="/5DF253FB/5DF53878" Ref="J6"  Part="1"
 F 0 "J6" H 2600 4525 50  0000 C CNN
-F 1 "DIN-5 MIDI Out" H 2600 4434 50  0000 C CNN
+F 1 "DIN-5 MIDI Through" H 2600 4434 50  0000 C CNN
 F 2 "JGP Footprints:5P180 DIN Socket" H 2600 4800 50  0001 C CNN
 F 3 "http://www.mouser.com/ds/2/18/40_c091_abd_e-75918.pdf" H 2600 4800 50  0001 C CNN

Commit message: Removing MIDI Through.
Parts:
- removed J6: DIN-5 MIDI Through, JGP Footprints:5P180 DIN Socket, symbol Connector:DIN-5_180degree
- removed R4, R7: 220, Resistor_THT:R_Axial_DIN0207_L6.3mm_D2.5mm_P10.16mm_Horizontal, symbol Device:R
Connections:
- net GND: now also U2.5, U2.9
- net MIDI_IN_TO_MCU: no longer U2.5
- net at U2.6: no longer U2.9
Changed lines of the file:
@@
-$EndComp
-$Comp
-L Connector:DIN-5_180degree J?
-U 1 1 5DF53878
-P 2600 4800
-AR Path="/5DF53878" Ref="J?"  Part="1"
-AR Path="/5DF253FB/5DF53878" Ref="J6"  Part="1"
-F 0 "J6" H 2600 4525 50  0000 C CNN
-F 1 "DIN-5 MIDI Through" H 2600 4434 50  0000 C CNN
-F 2 "JGP Footprints:5P180 DIN Socket" H 2600 4800 50  0001 C CNN
-F 3 "http://www.mouser.com/ds/2/18/40_c091_abd_e-75918.pdf" H 2600 4800 50  0001 C CNN
-	1    2600 4800
-	1    0    0    -1
 $EndComp
 $Comp
@@
 $EndComp
 $Comp
-L Device:R R7
-U 1 1 5E033CC2
-P 3300 4750
-F 0 "R7" V 3093 4750 50  0000 C CNN
-F 1 "220" V 3184 4750 50  0000 C CNN
-F 2 "Resistor_THT:R_Axial_DIN0207_L6.3mm_D2.5mm_P10.16mm_Horizontal" V 3230 4750 50  0001 C CNN
-F 3 "~" H 3300 4750 50  0001 C CNN
-F 4 "Stackpole Electronics Inc" H 3300 4750 50  0001 C CNN "Manufacturer"
-F 5 "CF14JT220R" H 3300 4750 50  0001 C CNN "PartNo"
-	1    3300 4750
-	0    1    1    0
-$EndComp
-$Comp
 L Device:R R9
 U 1 1 5E03403F
@@
 Wire Wire Line
 	5550 3750 5550 3500
-Wire Wire Line
-	5850 3750 5850 4750
-Wire Wire Line
-	5850 4750 5100 4750
-Wire Wire Line
-	5550 3750 5850 3750
 Connection ~ 5550 3750
 Wire Wire Line
-	4200 4750 4500 4750
-Wire Wire Line
 	4200 2650 4500 2650
 Wire Wire Line
 	3450 2650 3600 2650
 Wire Wire Line
-	3450 4750 3600 4750
-Wire Wire Line
 	2900 2600 3050 2600
 Wire Wire Line
@@
 Wire Wire Line
 	3050 2650 3150 2650
-Wire Wire Line
-	2900 4700 3050 4700
-Wire Wire Line
-	3050 4700 3050 4750
-Wire Wire Line
-	3050 4750 3150 4750
-$Comp
-L Device:R R4
-U 1 1 5E040B29
-P 2050 4450
-F 0 "R4" H 1980 4404 50  0000 R CNN
-F 1 "220" H 1980 4495 50  0000 R CNN
-F 2 "Resistor_THT:R_Axial_DIN0207_L6.3mm_D2.5mm_P10.16mm_Horizontal" V 1980 4450 50  0001 C CNN
-F 3 "~" H 2050 4450 50  0001 C CNN
-F 4 "Stackpole Electronics Inc" H 2050 4450 50  0001 C CNN "Manufacturer"
-F 5 "CF14JT220R" H 2050 4450 50  0001 C CNN "PartNo"
-	1    2050 4450
-	-1   0    0    1
-$EndComp
 $Comp
 L Device:R R3
@@
 	1    0    0    -1
 $EndComp
-$Comp
-L power:+5V #PWR?
-U 1 1 5E041A37
-P 2050 4200
-F 0 "#PWR?" H 2050 4050 50  0001 C CNN
-F 1 "+5V" H 2065 4373 50  0000 C CNN
-F 2 "" H 2050 4200 50  0001 C CNN
-F 3 "" H 2050 4200 50  0001 C CNN
-	1    2050 4200
-	1    0    0    -1
-$EndComp
 Wire Wire Line
 	2050 2100 2050 2200
@@
 Wire Wire Line
 	2050 2600 2300 2600
-Wire Wire Line
-	2050 4200 2050 4300
-Wire Wire Line
-	2050 4600 2050 4700
-Wire Wire Line
-	2050 4700 2300 4700
-Wire Wire Line
-	6200 3750 5850 3750
-Connection ~ 5850 3750
 Wire Wire Line
 	5100 2650 6150 2650
@@
 Wire Wire Line
 	8000 4150 8000 4200
-NoConn ~ 2900 4800
-NoConn ~ 2300 4800
 NoConn ~ 2300 3700
 NoConn ~ 2600 3400
@@
 	1    0    0    -1
 $EndComp
-$Comp
-L power:GND #PWR?
-U 1 1 5E06A577
-P 2800 4350
-F 0 "#PWR?" H 2800 4100 50  0001 C CNN
-F 1 "GND" H 2805 4177 50  0000 C CNN
-F 2 "" H 2800 4350 50  0001 C CNN
-F 3 "" H 2800 4350 50  0001 C CNN
-	1    2800 4350
-	1    0    0    -1
-$EndComp
-Wire Wire Line
-	2800 4350 2800 4300
-Wire Wire Line
-	2800 4300 2600 4300
-Wire Wire Line
-	2600 4300 2600 4500
 Wire Wire Line
 	2800 2200 2800 2150
@@
 Text Notes 5300 1650 0    100  ~ 20
 MIDI
+Wire Wire Line
+	5550 3750 6200 3750
+$Comp
+L power:GND #PWR?
+U 1 1 5E064042
+P 5250 5150
+F 0 "#PWR?" H 5250 4900 50  0001 C CNN
+F 1 "GND" H 5255 4977 50  0000 C CNN
+F 2 "" H 5250 5150 50  0001 C CNN
+F 3 "" H 5250 5150 50  0001 C CNN
+	1    5250 5150
+	1    0    0    -1
+$EndComp
+NoConn ~ 3600 4750
+NoConn ~ 4500 4750
+Wire Wire Line
+	5250 5150 5250 5050
+Wire Wire Line
+	5250 5050 5100 5050
+Wire Wire Line
+	4200 5050 4200 4750
+Wire Wire Line
+	5100 4750 5100 5050
+Connection ~ 5100 5050
+Wire Wire Line
+	5100 5050 4200 5050
 $EndSCHEMATC

Commit message: Updated BOM.
Parts:
- C1: Manufacturer (none) -> Vishay; PartNo (none) -> K104K15X7RF5TL2
- D1: value 1N148 -> 1N4148; Manufacturer (none) -> ON Semi; PartNo (none) -> 1N4148
- J4: value DIN-5 MIDI Out -> DIN-5 180 degree; Manufacturer (none) -> RS; PartNo (none) -> 491-087
- J5: value DIN-5 MIDI In -> DIN-5 180 degree; Manufacturer (none) -> RS; PartNo (none) -> 491-087; RS 491-087 -> (none)
Changed lines of the file:
@@
 AR Path="/5DF253FB/5DF5386C" Ref="J5"  Part="1"
 F 0 "J5" H 2600 3425 50  0000 C CNN
-F 1 "DIN-5 MIDI In" H 2600 3334 50  0000 C CNN
+F 1 "DIN-5 180 degree" H 2600 3334 50  0000 C CNN
 F 2 "JGP Footprints:5P180 DIN Socket" H 2600 3700 50  0001 C CNN
 F 3 "https://docs.rs-online.com/1ee9/0900766b81579be1.pdf" H 2600 3700 50  0001 C CNN
-F 4 "491-087" H 2600 3700 50  0001 C CNN "RS"
+F 4 "" H 2600 3700 50  0001 C CNN "RS"
+F 5 "RS" H 0   0   50  0001 C CNN "Manufacturer"
+F 6 "491-087" H 0   0   50  0001 C CNN "PartNo"
 	1    2600 3700
 	1    0    0    -1
@@
 AR Path="/5DF253FB/5DF53872" Ref="J4"  Part="1"
 F 0 "J4" H 2600 2425 50  0000 C CNN
-F 1 "DIN-5 MIDI Out" H 2600 2334 50  0000 C CNN
+F 1 "DIN-5 180 degree" H 2600 2334 50  0000 C CNN
 F 2 "JGP Footprints:5P180 DIN Socket" H 2600 2700 50  0001 C CNN
-F 3 "http://www.mouser.com/ds/2/18/40_c091_abd_e-75918.pdf" H 2600 2700 50  0001 C CNN
+F 3 "https://docs.rs-online.com/1ee9/0900766b81579be1.pdf" H 2600 2700 50  0001 C CNN
+F 4 "RS" H 0   0   50  0001 C CNN "Manufacturer"
+F 5 "491-087" H 0   0   50  0001 C CNN "PartNo"
 	1    2600 2700
 	1    0    0    -1
@@
 P 4250 3650
 F 0 "D1" V 4204 3729 50  0000 L CNN
-F 1 "1N148" V 4200 3300 50  0000 L CNN
+F 1 "1N4148" V 4200 3300 50  0000 L CNN
 F 2 "Diode_THT:D_DO-35_SOD27_P7.62mm_Horizontal" H 4250 3650 50  0001 C CNN
 F 3 "~" H 4250 3650 50  0001 C CNN
+F 4 "ON Semi" H 0   0   50  0001 C CNN "Manufacturer"
+F 5 "1N4148" H 0   0   50  0001 C CNN "PartNo"
 	1    4250 3650
 	0    1    1    0
@@
 F 2 "Capacitor_THT:C_Disc_D3.0mm_W2.0mm_P2.50mm" H 7538 3450 50  0001 C CNN
 F 3 "~" H 7500 3600 50  0001 C CNN
+F 4 "Vishay" H 0   0   50  0001 C CNN "Manufacturer"
+F 5 "K104K15X7RF5TL2" H 0   0   50  0001 C CNN "PartNo"
 	1    7500 3600
 	1    0    0    -1

Commit message: Add some extra explanatory notes.
Other:
- note added: "Provides two MIDI (Musical Instrument Digital Interface) ports. These function like a UART at a fixed 31,250 bps. One port is for MIDI In\nand the other is for MIDI Out. The MIDI standard requires the input is opto-isolated, so we use the 6N138. The Hex-Schmitt inverter is\nused as a level shifter and buffer."
- note removed: "MIDI"
Changed lines of the file:
@@
 EESchema Schematic File Version 4
-LIBS:neotron-32-cache
-EELAYER 26 0
+EELAYER 30 0
 EELAYER END
 $Descr A4 11693 8268
@@
 F 2 "JGP Footprints:5P180 DIN Socket" H 2600 3700 50  0001 C CNN
 F 3 "https://docs.rs-online.com/1ee9/0900766b81579be1.pdf" H 2600 3700 50  0001 C CNN
-F 5 "RS" H 0   0   50  0001 C CNN "Manufacturer"
-F 6 "491-087" H 0   0   50  0001 C CNN "PartNo"
+F 4 "RS" H 0   0   50  0001 C CNN "Manufacturer"
+F 5 "491-087" H 0   0   50  0001 C CNN "PartNo"
 	1    2600 3700
 	1    0    0    -1
@@
 Wire Wire Line
 	2600 2150 2600 2400
-Text Notes 5300 1650 0    100  ~ 20
-MIDI
 Wire Wire Line
 	5550 3750 6200 3750
@@
 Wire Wire Line
 	5100 5050 4200 5050
+Text Notes 550  7700 0    50   ~ 0
+Provides two MIDI (Musical Instrument Digital Interface) ports. These function like a UART at a fixed 31,250 bps. One port is for MIDI In\nand the other is for MIDI Out. The MIDI standard requires the input is opto-isolated, so we use the 6N138. The Hex-Schmitt inverter is\nused as a level shifter and buffer.
 $EndSCHEMATC

Commit message: Moved non-standard components into local libraries.
neotron-32.lib is the symbol library.
neotron-32.pretty is the footprint library.

Also swapped the DE9 and DB25 headers for IDC boxed versions. Involved
moving a resistor out of the way.

The Keystone 103 battery holder is a straight copy of the standard
footprint, but with the Courtyard removed to bypass the 'Courtyard is
not closed' DRC error.
Parts:
- J4, J5: footprint JGP Footprints:5P180 DIN Socket -> Neotron 32:5P180_DIN_Socket
Changed lines of the file:
@@
 F 0 "J5" H 2600 3425 50  0000 C CNN
 F 1 "DIN-5 180 degree" H 2600 3334 50  0000 C CNN
-F 2 "JGP Footprints:5P180 DIN Socket" H 2600 3700 50  0001 C CNN
+F 2 "Neotron 32:5P180_DIN_Socket" H 2600 3700 50  0001 C CNN
 F 3 "https://docs.rs-online.com/1ee9/0900766b81579be1.pdf" H 2600 3700 50  0001 C CNN
 F 4 "RS" H 0   0   50  0001 C CNN "Manufacturer"
@@
 F 0 "J4" H 2600 2425 50  0000 C CNN
 F 1 "DIN-5 180 degree" H 2600 2334 50  0000 C CNN
-F 2 "JGP Footprints:5P180 DIN Socket" H 2600 2700 50  0001 C CNN
+F 2 "Neotron 32:5P180_DIN_Socket" H 2600 2700 50  0001 C CNN
 F 3 "https://docs.rs-online.com/1ee9/0900766b81579be1.pdf" H 2600 2700 50  0001 C CNN
 F 4 "RS" H 0   0   50  0001 C CNN "Manufacturer"
