File: midi.sch (KiCad schematic (older format))
At the start: 11 parts, among them J4 DIN-5 180 degree, J5 DIN-5 180 degree, U2 74LS14, U3 6N138

Commit message: Replace PartNum with MPN so Kicost can see it.
Parts:
- C1: PartNo K104K15X7RF5TL2 -> (none); mpn (none) -> K104K15X7RF5TL2
- D1: PartNo 1N4148 -> (none); mpn (none) -> 1N4148
- J4, J5: PartNo 491-087 -> (none); mpn (none) -> 491-087
- R3, R5, R6: PartNo CF14JT220R -> (none); mpn (none) -> CF14JT220R
- R8: PartNo CF14JT10K0 -> (none); mpn (none) -> CF14JT10K0
- R9: PartNo CF14JT470R -> (none); mpn (none) -> CF14JT470R
- U2: PartNo SN74LS14N -> (none); mpn (none) -> SN74LS14N
- U3: PartNo 6N138 -> (none); mpn (none) -> 6N138
Changed lines of the file:
@@
 F 3 "https://docs.rs-online.com/1ee9/0900766b81579be1.pdf" H 2600 3700 50  0001 C CNN
 F 4 "RS" H 0   0   50  0001 C CNN "Manufacturer"
-F 5 "491-087" H 0   0   50  0001 C CNN "PartNo"
+F 5 "491-087" H 0   0   50  0001 C CNN "mpn"
 	1    2600 3700
 	1    0    0    -1
@@
 F 3 "https://docs.rs-online.com/1ee9/0900766b81579be1.pdf" H 2600 2700 50  0001 C CNN
 F 4 "RS" H 0   0   50  0001 C CNN "Manufacturer"
-F 5 "491-087" H 0   0   50  0001 C CNN "PartNo"
+F 5 "491-087" H 0   0   50  0001 C CNN "mpn"
 	1    2600 2700
 	1    0    0    -1
@@
 F 3 "https://media.digikey.com/pdf/Data%20Sheets/Lite-On%20PDFs/6N138-39%20Series.pdf" H 5190 3350 50  0001 C CNN
 F 4 "Lite-On Inc." H 4900 3650 50  0001 C CNN "Manufacturer"
-F 5 "6N138" H 4900 3650 50  0001 C CNN "PartNo"
+F 5 "6N138" H 4900 3650 50  0001 C CNN "mpn"
 	1    4900 3650
 	1    0    0    -1
@@
 F 3 "http://www.ti.com/lit/gpn/sn74LS14" H 3900 2650 50  0001 C CNN
 F 4 "Texas Instruments" H 3900 2650 50  0001 C CNN "Manufacturer"
-F 5 "SN74LS14N" H 3900 2650 50  0001 C CNN "PartNo"
+F 5 "SN74LS14N" H 3900 2650 50  0001 C CNN "mpn"
 	1    3900 2650
 	-1   0    0    1
@@
 F 3 "http://www.ti.com/lit/gpn/sn74LS14" H 4800 2650 50  0001 C CNN
 F 4 "Texas Instruments" H 4800 2650 50  0001 C CNN "Manufacturer"
-F 5 "SN74LS14N" H 4800 2650 50  0001 C CNN "PartNo"
+F 5 "SN74LS14N" H 4800 2650 50  0001 C CNN "mpn"
 	2    4800 2650
 	-1   0    0    1
@@
 F 3 "http://www.ti.com/lit/gpn/sn74LS14" H 4800 4750 50  0001 C CNN
 F 4 "Texas Instruments" H 4800 4750 50  0001 C CNN "Manufacturer"
-F 5 "SN74LS14N" H 4800 4750 50  0001 C CNN "PartNo"
+F 5 "SN74LS14N" H 4800 4750 50  0001 C CNN "mpn"
 	3    4800 4750
 	-1   0    0    1
@@
 F 3 "http://www.ti.com/lit/gpn/sn74LS14" H 3900 4750 50  0001 C CNN
 F 4 "Texas Instruments" H 3900 4750 50  0001 C CNN "Manufacturer"
-F 5 "SN74LS14N" H 3900 4750 50  0001 C CNN "PartNo"
+F 5 "SN74LS14N" H 3900 4750 50  0001 C CNN "mpn"
 	4    3900 4750
 	-1   0    0    1
@@
 F 3 "http://www.ti.com/lit/gpn/sn74LS14" H 8000 3600 50  0001 C CNN
 F 4 "Texas Instruments" H 8000 3600 50  0001 C CNN "Manufacturer"
-F 5 "SN74LS14N" H 8000 3600 50  0001 C CNN "PartNo"
+F 5 "SN74LS14N" H 8000 3600 50  0001 C CNN "mpn"
 	7    8000 3600
 	1    0    0    -1
@@
 F 3 "~" H 4250 3650 50  0001 C CNN
 F 4 "ON Semi" H 0   0   50  0001 C CNN "Manufacturer"
-F 5 "1N4148" H 0   0   50  0001 C CNN "PartNo"
+F 5 "1N4148" H 0   0   50  0001 C CNN "mpn"
 	1    4250 3650
 	0    1    1    0
@@
 F 3 "~" H 3200 3300 50  0001 C CNN
 F 4 "Stackpole Electronics Inc" H 3200 3300 50  0001 C CNN "Manufacturer"
-F 5 "CF14JT220R" H 3200 3300 50  0001 C CNN "PartNo"
+F 5 "CF14JT220R" H 3200 3300 50  0001 C CNN "mpn"
 	1    3200 3300
 	0    1    1    0
@@
 F 3 "~" H 3300 2650 50  0001 C CNN
 F 4 "Stackpole Electronics Inc" H 3300 2650 50  0001 C CNN "Manufacturer"
-F 5 "CF14JT220R" H 3300 2650 50  0001 C CNN "PartNo"
+F 5 "CF14JT220R" H 3300 2650 50  0001 C CNN "mpn"
 	1    3300 2650
 	0    1    1    0
@@
 F 3 "~" H 5550 3350 50  0001 C CNN
 F 4 "Stackpole Electronics Inc" H 5550 3350 50  0001 C CNN "Manufacturer"
-F 5 "CF14JT470R" H 5550 3350 50  0001 C CNN "PartNo"
+F 5 "CF14JT470R" H 5550 3350 50  0001 C CNN "mpn"
 	1    5550 3350
 	-1   0    0    1
@@
 F 3 "~" H 5400 4000 50  0001 C CNN
 F 4 "Stackpole Electronics Inc" H 5400 4000 50  0001 C CNN "Manufacturer"
-F 5 "CF14JT10K0" H 5400 4000 50  0001 C CNN "PartNo"
+F 5 "CF14JT10K0" H 5400 4000 50  0001 C CNN "mpn"
 	1    5400 4000
 	-1   0    0    1
@@
 F 3 "~" H 2050 2350 50  0001 C CNN
 F 4 "Stackpole Electronics Inc" H 2050 2350 50  0001 C CNN "Manufacturer"
-F 5 "CF14JT220R" H 2050 2350 50  0001 C CNN "PartNo"
+F 5 "CF14JT220R" H 2050 2350 50  0001 C CNN "mpn"
 	1    2050 2350
 	-1   0    0    1
@@
 F 3 "~" H 7500 3600 50  0001 C CNN
 F 4 "Vishay" H 0   0   50  0001 C CNN "Manufacturer"
-F 5 "K104K15X7RF5TL2" H 0   0   50  0001 C CNN "PartNo"
+F 5 "K104K15X7RF5TL2" H 0   0   50  0001 C CNN "mpn"
 	1    7500 3600
 	1    0    0    -1

Commit message: Tweaks to the BOM.
Marking parts as DNP=1 should stop them appearing in the BOM.
Also set multi-parts for ICs in sockets.
Parts:
- C1, D1, J4, J5, R3, R5, R6, R8, R9: DNP (none) -> 0
- U2: DNP (none) -> 0; Manufacturer Texas Instruments -> Texas Instruments;On Shore Technology; mpn SN74LS14N -> SN74LS14N;ED14DT
- U3: DNP (none) -> 0; Manufacturer Lite-On Inc. -> Lite-On Inc.;On Shore Technology; mpn 6N138 -> 6N138;ED08DT
Changed lines of the file:
@@
 F 4 "RS" H 0   0   50  0001 C CNN "Manufacturer"
 F 5 "491-087" H 0   0   50  0001 C CNN "mpn"
+F 6 "0" H 2600 3700 50  0001 C CNN "DNP"
 	1    2600 3700
 	1    0    0    -1
@@
 F 4 "RS" H 0   0   50  0001 C CNN "Manufacturer"
 F 5 "491-087" H 0   0   50  0001 C CNN "mpn"
+F 6 "0" H 2600 2700 50  0001 C CNN "DNP"
 	1    2600 2700
 	1    0    0    -1
@@
 F 2 "Package_DIP:DIP-8_W7.62mm" H 5190 3350 50  0001 C CNN
 F 3 "https://media.digikey.com/pdf/Data%20Sheets/Lite-On%20PDFs/6N138-39%20Series.pdf" H 5190 3350 50  0001 C CNN
-F 4 "Lite-On Inc." H 4900 3650 50  0001 C CNN "Manufacturer"
-F 5 "6N138" H 4900 3650 50  0001 C CNN "mpn"
+F 4 "Lite-On Inc.;On Shore Technology" H 4900 3650 50  0001 C CNN "Manufacturer"
+F 5 "6N138;ED08DT" H 4900 3650 50  0001 C CNN "mpn"
+F 6 "0" H 4900 3650 50  0001 C CNN "DNP"
 	1    4900 3650
 	1    0    0    -1
@@
 F 2 "Package_DIP:DIP-14_W7.62mm" H 3900 2650 50  0001 C CNN
 F 3 "http://www.ti.com/lit/gpn/sn74LS14" H 3900 2650 50  0001 C CNN
-F 4 "Texas Instruments" H 3900 2650 50  0001 C CNN "Manufacturer"
-F 5 "SN74LS14N" H 3900 2650 50  0001 C CNN "mpn"
+F 4 "Texas Instruments;On Shore Technology" H 3900 2650 50  0001 C CNN "Manufacturer"
+F 5 "SN74LS14N;ED14DT" H 3900 2650 50  0001 C CNN "mpn"
+F 6 "0" H 3900 2650 50  0001 C CNN "DNP"
 	1    3900 2650
 	-1   0    0    1
@@
 F 2 "Package_DIP:DIP-14_W7.62mm" H 4800 2650 50  0001 C CNN
 F 3 "http://www.ti.com/lit/gpn/sn74LS14" H 4800 2650 50  0001 C CNN
-F 4 "Texas Instruments" H 4800 2650 50  0001 C CNN "Manufacturer"
-F 5 "SN74LS14N" H 4800 2650 50  0001 C CNN "mpn"
+F 4 "Texas Instruments;On Shore Technology" H 4800 2650 50  0001 C CNN "Manufacturer"
+F 5 "SN74LS14N;ED14DT" H 4800 2650 50  0001 C CNN "mpn"
+F 6 "0" H 4800 2650 50  0001 C CNN "DNP"
 	2    4800 2650
 	-1   0    0    1
@@
 F 2 "Package_DIP:DIP-14_W7.62mm" H 4800 4750 50  0001 C CNN
 F 3 "http://www.ti.com/lit/gpn/sn74LS14" H 4800 4750 50  0001 C CNN
-F 4 "Texas Instruments" H 4800 4750 50  0001 C CNN "Manufacturer"
-F 5 "SN74LS14N" H 4800 4750 50  0001 C CNN "mpn"
+F 4 "Texas Instruments;On Shore Technology" H 4800 4750 50  0001 C CNN "Manufacturer"
+F 5 "SN74LS14N;ED14DT" H 4800 4750 50  0001 C CNN "mpn"
+F 6 "0" H 4800 4750 50  0001 C CNN "DNP"
 	3    4800 4750
 	-1   0    0    1
@@
 F 2 "Package_DIP:DIP-14_W7.62mm" H 3900 4750 50  0001 C CNN
 F 3 "http://www.ti.com/lit/gpn/sn74LS14" H 3900 4750 50  0001 C CNN
-F 4 "Texas Instruments" H 3900 4750 50  0001 C CNN "Manufacturer"
-F 5 "SN74LS14N" H 3900 4750 50  0001 C CNN "mpn"
+F 4 "Texas Instruments;On Shore Technology" H 3900 4750 50  0001 C CNN "Manufacturer"
+F 5 "SN74LS14N;ED14DT" H 3900 4750 50  0001 C CNN "mpn"
+F 6 "0" H 3900 4750 50  0001 C CNN "DNP"
 	4    3900 4750
 	-1   0    0    1
@@
 F 2 "Package_DIP:DIP-14_W7.62mm" H 8000 3600 50  0001 C CNN
 F 3 "http://www.ti.com/lit/gpn/sn74LS14" H 8000 3600 50  0001 C CNN
-F 4 "Texas Instruments" H 8000 3600 50  0001 C CNN "Manufacturer"
-F 5 "SN74LS14N" H 8000 3600 50  0001 C CNN "mpn"
+F 4 "Texas Instruments;On Shore Technology" H 8000 3600 50  0001 C CNN "Manufacturer"
+F 5 "SN74LS14N;ED14DT" H 8000 3600 50  0001 C CNN "mpn"
+F 6 "0" H 8000 3600 50  0001 C CNN "DNP"
 	7    8000 3600
 	1    0    0    -1
@@
 F 4 "ON Semi" H 0   0   50  0001 C CNN "Manufacturer"
 F 5 "1N4148" H 0   0   50  0001 C CNN "mpn"
+F 6 "0" H 4250 3650 50  0001 C CNN "DNP"
 	1    4250 3650
 	0    1    1    0
@@
 F 4 "Stackpole Electronics Inc" H 3200 3300 50  0001 C CNN "Manufacturer"
 F 5 "CF14JT220R" H 3200 3300 50  0001 C CNN "mpn"
+F 6 "0" H 3200 3300 50  0001 C CNN "DNP"
 	1    3200 3300
 	0    1    1    0
@@
 F 4 "Stackpole Electronics Inc" H 3300 2650 50  0001 C CNN "Manufacturer"
 F 5 "CF14JT220R" H 3300 2650 50  0001 C CNN "mpn"
+F 6 "0" H 3300 2650 50  0001 C CNN "DNP"
 	1    3300 2650
 	0    1    1    0
@@
 F 4 "Stackpole Electronics Inc" H 5550 3350 50  0001 C CNN "Manufacturer"
 F 5 "CF14JT470R" H 5550 3350 50  0001 C CNN "mpn"
+F 6 "0" H 5550 3350 50  0001 C CNN "DNP"
 	1    5550 3350
 	-1   0    0    1
@@
 F 4 "Stackpole Electronics Inc" H 5400 4000 50  0001 C CNN "Manufacturer"
 F 5 "CF14JT10K0" H 5400 4000 50  0001 C CNN "mpn"
+F 6 "0" H 5400 4000 50  0001 C CNN "DNP"
 	1    5400 4000
 	-1   0    0    1
@@
 F 4 "Stackpole Electronics Inc" H 2050 2350 50  0001 C CNN "Manufacturer"
 F 5 "CF14JT220R" H 2050 2350 50  0001 C CNN "mpn"
+F 6 "0" H 2050 2350 50  0001 C CNN "DNP"
 	1    2050 2350
 	-1   0    0    1
@@
 F 4 "Vishay" H 0   0   50  0001 C CNN "Manufacturer"
 F 5 "K104K15X7RF5TL2" H 0   0   50  0001 C CNN "mpn"
+F 6 "0" H 7500 3600 50  0001 C CNN "DNP"
 	1    7500 3600
 	1    0    0    -1
