File: audio.sch (KiCad schematic (older format))
At the start: 10 parts, among them J7 3.5mm Audio Jack TRS, J8 Conn_01x03_Male

Commit message: Adding MPNs.
Parts:
- R10, R11: Manufacturer (none) -> Stackpole Electronics Inc; PartNo (none) -> CF14JT270R
- R12, R13: Manufacturer (none) -> Stackpole Electronics Inc; PartNo (none) -> CF14JT150R
Changed lines of the file:
@@
 F 2 "Resistor_THT:R_Axial_DIN0207_L6.3mm_D2.5mm_P10.16mm_Horizontal" V 5530 3400 50  0001 C CNN
 F 3 "~" H 5600 3400 50  0001 C CNN
+F 4 "Stackpole Electronics Inc" H 5600 3400 50  0001 C CNN "Manufacturer"
+F 5 "CF14JT150R" H 5600 3400 50  0001 C CNN "PartNo"
 	1    5600 3400
 	1    0    0    -1
@@
 F 2 "Resistor_THT:R_Axial_DIN0207_L6.3mm_D2.5mm_P10.16mm_Horizontal" V 5530 4100 50  0001 C CNN
 F 3 "~" H 5600 4100 50  0001 C CNN
+F 4 "Stackpole Electronics Inc" H 5600 4100 50  0001 C CNN "Manufacturer"
+F 5 "CF14JT150R" H 5600 4100 50  0001 C CNN "PartNo"
 	1    5600 4100
 	1    0    0    -1
@@
 F 2 "Resistor_THT:R_Axial_DIN0207_L6.3mm_D2.5mm_P10.16mm_Horizontal" V 4630 3900 50  0001 C CNN
 F 3 "~" H 4700 3900 50  0001 C CNN
+F 4 "Stackpole Electronics Inc" H 4700 3900 50  0001 C CNN "Manufacturer"
+F 5 "CF14JT270R" H 4700 3900 50  0001 C CNN "PartNo"
 	1    4700 3900
 	0    1    1    0
@@
 F 2 "Resistor_THT:R_Axial_DIN0207_L6.3mm_D2.5mm_P10.16mm_Horizontal" V 4630 3200 50  0001 C CNN
 F 3 "~" H 4700 3200 50  0001 C CNN
+F 4 "Stackpole Electronics Inc" H 4700 3200 50  0001 C CNN "Manufacturer"
+F 5 "CF14JT270R" H 4700 3200 50  0001 C CNN "PartNo"
 	1    4700 3200
 	0    1    1    0

Commit message: Updated BOM.
Parts:
- C2, C3: Manufacturer (none) -> Vishay; PartNo (none) -> K333K15X7RF5TL2
- C4, C5: Manufacturer (none) -> Vishay; PartNo (none) -> MAL203858109E3
- J7: Manufacturer (none) -> CUI; PartNo (none) -> SJ1-3533NG
Changed lines of the file:
@@
 F 2 "Connector_Audio:Jack_3.5mm_CUI_SJ1-3533NG_Horizontal" H 7100 4150 50  0001 C CNN
 F 3 "~" H 7100 4150 50  0001 C CNN
+F 4 "CUI" H 0   0   50  0001 C CNN "Manufacturer"
+F 5 "SJ1-3533NG " H 0   0   50  0001 C CNN "PartNo"
 	1    7100 4150
 	-1   0    0    1
@@
 F 2 "Connector_PinHeader_2.54mm:PinHeader_1x03_P2.54mm_Vertical" H 7250 3300 50  0001 C CNN
 F 3 "~" H 7250 3300 50  0001 C CNN
+F 4 "~" H 0   0   50  0001 C CNN "Manufacturer"
+F 5 "~" H 0   0   50  0001 C CNN "PartNo"
 	1    7250 3300
 	-1   0    0    1
@@
 F 2 "Capacitor_THT:CP_Radial_D6.3mm_P2.50mm" H 5938 3050 50  0001 C CNN
 F 3 "~" H 5900 3200 50  0001 C CNN
+F 4 "Vishay" H 0   0   50  0001 C CNN "Manufacturer"
+F 5 "MAL203858109E3" H 0   0   50  0001 C CNN "PartNo"
 	1    5900 3200
 	0    -1   -1   0
@@
 F 2 "Capacitor_THT:CP_Radial_D6.3mm_P2.50mm" H 5938 3750 50  0001 C CNN
 F 3 "~" H 5900 3900 50  0001 C CNN
+F 4 "Vishay" H 0   0   50  0001 C CNN "Manufacturer"
+F 5 "MAL203858109E3" H 0   0   50  0001 C CNN "PartNo"
 	1    5900 3900
 	0    -1   -1   0
@@
 F 2 "Capacitor_THT:C_Disc_D3.0mm_W2.0mm_P2.50mm" H 5188 3950 50  0001 C CNN
 F 3 "~" H 5150 4100 50  0001 C CNN
+F 4 "Vishay" H 0   0   50  0001 C CNN "Manufacturer"
+F 5 "K333K15X7RF5TL2" H 0   0   50  0001 C CNN "PartNo"
 	1    5150 4100
 	-1   0    0    1
@@
 F 2 "Capacitor_THT:C_Disc_D3.0mm_W2.0mm_P2.50mm" H 5188 3250 50  0001 C CNN
 F 3 "~" H 5150 3400 50  0001 C CNN
+F 4 "Vishay" H 0   0   50  0001 C CNN "Manufacturer"
+F 5 "K333K15X7RF5TL2" H 0   0   50  0001 C CNN "PartNo"
 	1    5150 3400
 	-1   0    0    1

Commit message: Add some extra explanatory notes.
Other:
- note added: "The filter is very similar to that on a Raspberry Pi. You will need to connect some amplified speakers with their own volume control, as the\noutput is pretty weak.\n\nSet the jumper to 1-2 to send the Left Channel audio from the CPU to both the Left (Tip) and Right (Ring) outputs on the 3.5mm Jack.\n\nSet the jumper to 2-3 to send the Left Channel audio from the CPU to both the Left (Tip) output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"
- note removed: "Audio"
Changed lines of the file:
@@
 EESchema Schematic File Version 4
-LIBS:neotron-32-cache
-EELAYER 26 0
+EELAYER 30 0
 EELAYER END
 $Descr A4 11693 8268
@@
 Wire Wire Line
 	6350 3300 6350 4150
-Text Notes 5250 2100 0    100  ~ 20
-Audio
+Text Notes 550  7700 0    50   ~ 0
+The filter is very similar to that on a Raspberry Pi. You will need to connect some amplified speakers with their own volume control, as the\noutput is pretty weak.\n\nSet the jumper to 1-2 to send the Left Channel audio from the CPU to both the Left (Tip) and Right (Ring) outputs on the 3.5mm Jack.\n\nSet the jumper to 2-3 to send the Left Channel audio from the CPU to both the Left (Tip) output on the 3.5mm jack and the Right Channel\naudio from the CPU to the right (ring) channel on the 3.5mm Jack.\n\n
 $EndSCHEMATC
