File: audio.sch (KiCad schematic (older format))
At the start: 10 parts, among them J7 3.5mm Audio Jack TRS, J8 Conn_01x03_Male

Commit message: Replace PartNum with MPN so Kicost can see it.
Parts:
- C2, C3: PartNo K333K15X7RF5TL2 -> (none); mpn (none) -> K333K15X7RF5TL2
- C4, C5: PartNo MAL203858109E3 -> (none); mpn (none) -> MAL203858109E3
- J7: PartNo SJ1-3533NG -> (none); mpn (none) -> SJ1-3533NG
- R10, R11: PartNo CF14JT270R -> (none); mpn (none) -> CF14JT270R
- R12, R13: PartNo CF14JT150R -> (none); mpn (none) -> CF14JT150R
Changed lines of the file:
@@
 F 3 "~" H 7100 4150 50  0001 C CNN
 F 4 "CUI" H 0   0   50  0001 C CNN "Manufacturer"
-F 5 "SJ1-3533NG " H 0   0   50  0001 C CNN "PartNo"
+F 5 "SJ1-3533NG " H 0   0   50  0001 C CNN "mpn"
 	1    7100 4150
 	-1   0    0    1
@@
 F 3 "~" H 7250 3300 50  0001 C CNN
 F 4 "~" H 0   0   50  0001 C CNN "Manufacturer"
-F 5 "~" H 0   0   50  0001 C CNN "PartNo"
+F 5 "~" H 0   0   50  0001 C CNN "mpn"
 	1    7250 3300
 	-1   0    0    1
@@
 F 3 "~" H 5900 3200 50  0001 C CNN
 F 4 "Vishay" H 0   0   50  0001 C CNN "Manufacturer"
-F 5 "MAL203858109E3" H 0   0   50  0001 C CNN "PartNo"
+F 5 "MAL203858109E3" H 0   0   50  0001 C CNN "mpn"
 	1    5900 3200
 	0    -1   -1   0
@@
 F 3 "~" H 5900 3900 50  0001 C CNN
 F 4 "Vishay" H 0   0   50  0001 C CNN "Manufacturer"
-F 5 "MAL203858109E3" H 0   0   50  0001 C CNN "PartNo"
+F 5 "MAL203858109E3" H 0   0   50  0001 C CNN "mpn"
 	1    5900 3900
 	0    -1   -1   0
@@
 F 3 "~" H 5600 3400 50  0001 C CNN
 F 4 "Stackpole Electronics Inc" H 5600 3400 50  0001 C CNN "Manufacturer"
-F 5 "CF14JT150R" H 5600 3400 50  0001 C CNN "PartNo"
+F 5 "CF14JT150R" H 5600 3400 50  0001 C CNN "mpn"
 	1    5600 3400
 	1    0    0    -1
@@
 F 3 "~" H 5600 4100 50  0001 C CNN
 F 4 "Stackpole Electronics Inc" H 5600 4100 50  0001 C CNN "Manufacturer"
-F 5 "CF14JT150R" H 5600 4100 50  0001 C CNN "PartNo"
+F 5 "CF14JT150R" H 5600 4100 50  0001 C CNN "mpn"
 	1    5600 4100
 	1    0    0    -1
@@
 F 3 "~" H 4700 3900 50  0001 C CNN
 F 4 "Stackpole Electronics Inc" H 4700 3900 50  0001 C CNN "Manufacturer"
-F 5 "CF14JT270R" H 4700 3900 50  0001 C CNN "PartNo"
+F 5 "CF14JT270R" H 4700 3900 50  0001 C CNN "mpn"
 	1    4700 3900
 	0    1    1    0
@@
 F 3 "~" H 4700 3200 50  0001 C CNN
 F 4 "Stackpole Electronics Inc" H 4700 3200 50  0001 C CNN "Manufacturer"
-F 5 "CF14JT270R" H 4700 3200 50  0001 C CNN "PartNo"
+F 5 "CF14JT270R" H 4700 3200 50  0001 C CNN "mpn"
 	1    4700 3200
 	0    1    1    0
@@
 F 3 "~" H 5150 4100 50  0001 C CNN
 F 4 "Vishay" H 0   0   50  0001 C CNN "Manufacturer"
-F 5 "K333K15X7RF5TL2" H 0   0   50  0001 C CNN "PartNo"
+F 5 "K333K15X7RF5TL2" H 0   0   50  0001 C CNN "mpn"
 	1    5150 4100
 	-1   0    0    1
@@
 F 3 "~" H 5150 3400 50  0001 C CNN
 F 4 "Vishay" H 0   0   50  0001 C CNN "Manufacturer"
-F 5 "K333K15X7RF5TL2" H 0   0   50  0001 C CNN "PartNo"
+F 5 "K333K15X7RF5TL2" H 0   0   50  0001 C CNN "mpn"
 	1    5150 3400
 	-1   0    0    1

Commit message: Tweaks to the BOM.
Marking parts as DNP=1 should stop them appearing in the BOM.
Also set multi-parts for ICs in sockets.
Parts:
- C2, C3, C4, C5, J7, J8, R10, R11, R12, R13: DNP (none) -> 0
Changed lines of the file:
@@
 F 4 "CUI" H 0   0   50  0001 C CNN "Manufacturer"
 F 5 "SJ1-3533NG " H 0   0   50  0001 C CNN "mpn"
+F 6 "0" H 7100 4150 50  0001 C CNN "DNP"
 	1    7100 4150
 	-1   0    0    1
@@
 F 4 "~" H 0   0   50  0001 C CNN "Manufacturer"
 F 5 "~" H 0   0   50  0001 C CNN "mpn"
+F 6 "0" H 7250 3300 50  0001 C CNN "DNP"
 	1    7250 3300
 	-1   0    0    1
@@
 F 4 "Vishay" H 0   0   50  0001 C CNN "Manufacturer"
 F 5 "MAL203858109E3" H 0   0   50  0001 C CNN "mpn"
+F 6 "0" H 5900 3200 50  0001 C CNN "DNP"
 	1    5900 3200
 	0    -1   -1   0
@@
 F 4 "Vishay" H 0   0   50  0001 C CNN "Manufacturer"
 F 5 "MAL203858109E3" H 0   0   50  0001 C CNN "mpn"
+F 6 "0" H 5900 3900 50  0001 C CNN "DNP"
 	1    5900 3900
 	0    -1   -1   0
@@
 F 4 "Stackpole Electronics Inc" H 5600 3400 50  0001 C CNN "Manufacturer"
 F 5 "CF14JT150R" H 5600 3400 50  0001 C CNN "mpn"
+F 6 "0" H 5600 3400 50  0001 C CNN "DNP"
 	1    5600 3400
 	1    0    0    -1
@@
 F 4 "Stackpole Electronics Inc" H 5600 4100 50  0001 C CNN "Manufacturer"
 F 5 "CF14JT150R" H 5600 4100 50  0001 C CNN "mpn"
+F 6 "0" H 5600 4100 50  0001 C CNN "DNP"
 	1    5600 4100
 	1    0    0    -1
@@
 F 4 "Stackpole Electronics Inc" H 4700 3900 50  0001 C CNN "Manufacturer"
 F 5 "CF14JT270R" H 4700 3900 50  0001 C CNN "mpn"
+F 6 "0" H 4700 3900 50  0001 C CNN "DNP"
 	1    4700 3900
 	0    1    1    0
@@
 F 4 "Stackpole Electronics Inc" H 4700 3200 50  0001 C CNN "Manufacturer"
 F 5 "CF14JT270R" H 4700 3200 50  0001 C CNN "mpn"
+F 6 "0" H 4700 3200 50  0001 C CNN "DNP"
 	1    4700 3200
 	0    1    1    0
@@
 F 4 "Vishay" H 0   0   50  0001 C CNN "Manufacturer"
 F 5 "K333K15X7RF5TL2" H 0   0   50  0001 C CNN "mpn"
+F 6 "0" H 5150 4100 50  0001 C CNN "DNP"
 	1    5150 4100
 	-1   0    0    1
@@
 F 4 "Vishay" H 0   0   50  0001 C CNN "Manufacturer"
 F 5 "K333K15X7RF5TL2" H 0   0   50  0001 C CNN "mpn"
+F 6 "0" H 5150 3400 50  0001 C CNN "DNP"
 	1    5150 3400
 	-1   0    0    1
