File: rtc.sch (KiCad schematic (older format))
At the start: 6 parts, among them U7 MCP7940N-xP, Y1 32,768 Hz

Commit message: Replaced broken Keystone 103 footprint with edited one.
Stops annoying DRC error.
Parts:
- BT1: footprint Battery:BatteryHolder_Keystone_103_1x20mm -> JGP Footprints:BatteryHolder_Keystone_103_1x20mm
Changed lines of the file:
@@
 F 0 "BT1" H 6418 3496 50  0000 L CNN
 F 1 "CR2023" H 6418 3405 50  0000 L CNN
-F 2 "Battery:BatteryHolder_Keystone_103_1x20mm" V 6300 3460 50  0001 C CNN
+F 2 "JGP Footprints:BatteryHolder_Keystone_103_1x20mm" V 6300 3460 50  0001 C CNN
 F 3 "~" V 6300 3460 50  0001 C CNN
 	1    6300 3400

Commit message: Adding MPNs.
Parts:
- BT1: value CR2023 -> CR2032; Manufacturer (none) -> Keystone; PartNo (none) -> 103
- U7: Manufacturer (none) -> Microchip; PartNo (none) -> MCP7940N-I/P
- Y1: Manufacturer (none) -> Citizen; PartNo (none) -> CFS-20632768DZBB
Changed lines of the file:
@@
 F 2 "Package_DIP:DIP-8_W7.62mm" H 4950 3350 50  0001 C CNN
 F 3 "http://ww1.microchip.com/downloads/en/DeviceDoc/20005010F.pdf" H 4950 3350 50  0001 C CNN
+F 4 "Microchip" H 4950 3350 50  0001 C CNN "Manufacturer"
+F 5 "MCP7940N-I/P" H 4950 3350 50  0001 C CNN "PartNo"
 	1    4950 3350
 	1    0    0    -1
@@
 P 6300 3400
 F 0 "BT1" H 6418 3496 50  0000 L CNN
-F 1 "CR2023" H 6418 3405 50  0000 L CNN
+F 1 "CR2032" H 6418 3405 50  0000 L CNN
 F 2 "JGP Footprints:BatteryHolder_Keystone_103_1x20mm" V 6300 3460 50  0001 C CNN
 F 3 "~" V 6300 3460 50  0001 C CNN
+F 4 "Keystone" H 6300 3400 50  0001 C CNN "Manufacturer"
+F 5 "103" H 6300 3400 50  0001 C CNN "PartNo"
 	1    6300 3400
 	1    0    0    -1
@@
 F 3 "http://cfd.citizen.co.jp/english/prod-tech/product/pdf/datasheet_TF/CFS-206_CFS-145_E.pdf" H 5550 3350 50  0001 C CNN
 F 4 "CFS-20632768DZBB" V 5550 3350 50  0001 C CNN "Digikey"
+F 5 "Citizen" H 5550 3350 50  0001 C CNN "Manufacturer"
+F 6 "CFS-20632768DZBB " H 5550 3350 50  0001 C CNN "PartNo"
 	1    5550 3350
 	0    1    1    0

Commit message: Updated BOM.
Parts:
- C21, C22: Manufacturer (none) -> TDK; PartNo (none) -> FG18C0G1H060DNT06
- C23: Manufacturer (none) -> Vishay; PartNo (none) -> K104K15X7RF5TL2
- Y1: Digikey CFS-20632768DZBB -> (none)
Changed lines of the file:
@@
 F 2 "Capacitor_THT:C_Disc_D3.0mm_W2.0mm_P2.50mm" H 7088 3200 50  0001 C CNN
 F 3 "~" H 7050 3350 50  0001 C CNN
+F 4 "Vishay" H 0   0   50  0001 C CNN "Manufacturer"
+F 5 "K104K15X7RF5TL2" H 0   0   50  0001 C CNN "PartNo"
 	1    7050 3350
 	1    0    0    -1
@@
 F 2 "Crystal:Crystal_C26-LF_D2.1mm_L6.5mm_Horizontal" H 5550 3350 50  0001 C CNN
 F 3 "http://cfd.citizen.co.jp/english/prod-tech/product/pdf/datasheet_TF/CFS-206_CFS-145_E.pdf" H 5550 3350 50  0001 C CNN
-F 4 "CFS-20632768DZBB" V 5550 3350 50  0001 C CNN "Digikey"
+F 4 "" V 5550 3350 50  0001 C CNN "Digikey"
 F 5 "Citizen" H 5550 3350 50  0001 C CNN "Manufacturer"
 F 6 "CFS-20632768DZBB " H 5550 3350 50  0001 C CNN "PartNo"
@@
 F 2 "Capacitor_THT:C_Disc_D3.0mm_W2.0mm_P2.50mm" H 5588 2800 50  0001 C CNN
 F 3 "~" H 5550 2950 50  0001 C CNN
+F 4 "TDK" H 0   0   50  0001 C CNN "Manufacturer"
+F 5 "FG18C0G1H060DNT06" H 0   0   50  0001 C CNN "PartNo"
 	1    5550 2950
 	1    0    0    -1
@@
 F 2 "Capacitor_THT:C_Disc_D3.0mm_W2.0mm_P2.50mm" H 5588 3600 50  0001 C CNN
 F 3 "~" H 5550 3750 50  0001 C CNN
+F 4 "TDK" H 0   0   50  0001 C CNN "Manufacturer"
+F 5 "FG18C0G1H060DNT06" H 0   0   50  0001 C CNN "PartNo"
 	1    5550 3750
 	1    0    0    -1

Commit message: Add some extra explanatory notes.
Other:
- note added: "The Real-Time Clock uses an (optional) 3V coin cell as battery backup.\n\nIt appears on the I2C bus as 7-bit address 0x6F."
- note removed: "Real Time Clock"
Changed lines of the file:
@@
 EESchema Schematic File Version 4
-LIBS:neotron-32-cache
-EELAYER 26 0
+EELAYER 30 0
 EELAYER END
 $Descr A4 11693 8268
@@
 F 2 "Crystal:Crystal_C26-LF_D2.1mm_L6.5mm_Horizontal" H 5550 3350 50  0001 C CNN
 F 3 "http://cfd.citizen.co.jp/english/prod-tech/product/pdf/datasheet_TF/CFS-206_CFS-145_E.pdf" H 5550 3350 50  0001 C CNN
-F 5 "Citizen" H 5550 3350 50  0001 C CNN "Manufacturer"
-F 6 "CFS-20632768DZBB " H 5550 3350 50  0001 C CNN "PartNo"
+F 4 "Citizen" H 5550 3350 50  0001 C CNN "Manufacturer"
+F 5 "CFS-20632768DZBB " H 5550 3350 50  0001 C CNN "PartNo"
 	1    5550 3350
 	0    1    1    0
@@
 Wire Wire Line
 	6300 3150 6300 3200
-Text Notes 5050 2150 0    100  ~ 20
-Real Time Clock
+Text Notes 550  7700 0    50   Italic 0
+The Real-Time Clock uses an (optional) 3V coin cell as battery backup.\n\nIt appears on the I2C bus as 7-bit address 0x6F.
 $EndSCHEMATC

Commit message: Moved non-standard components into local libraries.
neotron-32.lib is the symbol library.
neotron-32.pretty is the footprint library.

Also swapped the DE9 and DB25 headers for IDC boxed versions. Involved
moving a resistor out of the way.

The Keystone 103 battery holder is a straight copy of the standard
footprint, but with the Courtyard removed to bypass the 'Courtyard is
not closed' DRC error.
Parts:
- BT1: footprint JGP Footprints:BatteryHolder_Keystone_103_1x20mm -> Neotron 32:BatteryHolder_Keystone_103_1x20mm
Changed lines of the file:
@@
 F 0 "BT1" H 6418 3496 50  0000 L CNN
 F 1 "CR2032" H 6418 3405 50  0000 L CNN
-F 2 "JGP Footprints:BatteryHolder_Keystone_103_1x20mm" V 6300 3460 50  0001 C CNN
+F 2 "Neotron 32:BatteryHolder_Keystone_103_1x20mm" V 6300 3460 50  0001 C CNN
 F 3 "~" V 6300 3460 50  0001 C CNN
 F 4 "Keystone" H 6300 3400 50  0001 C CNN "Manufacturer"
