File: vga.sch (KiCad schematic (older format))
At the start: 7 parts, among them J17 DB15HD_Female

Commit message: Adding MPNs.
Parts:
- J17: Manufacturer (none) -> Amphenol; PartNo (none) -> ICD15S13E4GV00LF
- R22, R23, R24: Manufacturer (none) -> Stackpole Electronics Inc; PartNo (none) -> CF14JT330R
- R26, R27: Manufacturer (none) -> Stackpole Electronics Inc; PartNo (none) -> CF14JT470R
Changed lines of the file:
@@
 F 3 "https://www.amphenol-icc.com/media/wysiwyg/files/drawing/c-cd-0012.pdf" H 4600 3650 50  0001 C CNN
 F 4 "609-5180-ND" H 5550 3250 50  0001 C CNN "Digikey"
+F 5 "Amphenol" H 5550 3250 50  0001 C CNN "Manufacturer"
+F 6 "ICD15S13E4GV00LF" H 5550 3250 50  0001 C CNN "PartNo"
 	1    5550 3250
 	1    0    0    -1
@@
 F 2 "Resistor_THT:R_Axial_DIN0207_L6.3mm_D2.5mm_P10.16mm_Horizontal" V 6030 3450 50  0001 C CNN
 F 3 "~" H 6100 3450 50  0001 C CNN
+F 4 "Stackpole Electronics Inc" H 6100 3450 50  0001 C CNN "Manufacturer"
+F 5 "CF14JT470R" H 6100 3450 50  0001 C CNN "PartNo"
 	1    6100 3450
 	0    1    1    0
@@
 F 2 "Resistor_THT:R_Axial_DIN0207_L6.3mm_D2.5mm_P10.16mm_Horizontal" V 6030 3250 50  0001 C CNN
 F 3 "~" H 6100 3250 50  0001 C CNN
+F 4 "Stackpole Electronics Inc" H 6100 3250 50  0001 C CNN "Manufacturer"
+F 5 "CF14JT470R" H 6100 3250 50  0001 C CNN "PartNo"
 	1    6100 3250
 	0    1    1    0
@@
 F 2 "Resistor_THT:R_Axial_DIN0207_L6.3mm_D2.5mm_P10.16mm_Horizontal" V 4930 2850 50  0001 C CNN
 F 3 "~" H 5000 2850 50  0001 C CNN
+F 4 "Stackpole Electronics Inc" H 5000 2850 50  0001 C CNN "Manufacturer"
+F 5 "CF14JT330R" H 5000 2850 50  0001 C CNN "PartNo"
 	1    5000 2850
 	0    1    1    0
@@
 F 2 "Resistor_THT:R_Axial_DIN0207_L6.3mm_D2.5mm_P10.16mm_Horizontal" V 4930 3050 50  0001 C CNN
 F 3 "~" H 5000 3050 50  0001 C CNN
+F 4 "Stackpole Electronics Inc" H 5000 3050 50  0001 C CNN "Manufacturer"
+F 5 "CF14JT330R" H 5000 3050 50  0001 C CNN "PartNo"
 	1    5000 3050
 	0    1    1    0
@@
 F 2 "Resistor_THT:R_Axial_DIN0207_L6.3mm_D2.5mm_P10.16mm_Horizontal" V 4930 3250 50  0001 C CNN
 F 3 "~" H 5000 3250 50  0001 C CNN
+F 4 "Stackpole Electronics Inc" H 5000 3250 50  0001 C CNN "Manufacturer"
+F 5 "CF14JT330R" H 5000 3250 50  0001 C CNN "PartNo"
 	1    5000 3250
 	0    1    1    0

Commit message: Updated BOM.
Parts:
- J17: Digikey 609-5180-ND -> (none)
Changed lines of the file:
@@
 F 2 "Connector_Dsub:DSUB-15-HD_Female_Horizontal_P2.29x1.98mm_EdgePinOffset3.03mm_Housed_MountingHolesOffset4.94mm" H 4600 3650 50  0001 C CNN
 F 3 "https://www.amphenol-icc.com/media/wysiwyg/files/drawing/c-cd-0012.pdf" H 4600 3650 50  0001 C CNN
-F 4 "609-5180-ND" H 5550 3250 50  0001 C CNN "Digikey"
+F 4 "" H 5550 3250 50  0001 C CNN "Digikey"
 F 5 "Amphenol" H 5550 3250 50  0001 C CNN "Manufacturer"
 F 6 "ICD15S13E4GV00LF" H 5550 3250 50  0001 C CNN "PartNo"
@@
 F 2 "Resistor_THT:R_Axial_DIN0207_L6.3mm_D2.5mm_P10.16mm_Horizontal" V 5830 3950 50  0001 C CNN
 F 3 "~" H 5900 3950 50  0001 C CNN
+F 4 "~" H 0   0   50  0001 C CNN "Manufacturer"
+F 5 "~" H 0   0   50  0001 C CNN "PartNo"
 	1    5900 3950
 	0    1    1    0

Commit message: Add some extra explanatory notes.
Other:
- note added: "The VGA output is driven directly from the GPIO pins using a resistive divider. The output impedance is therefore all wrong. Best results\nare with an LCD monitor and a short VGA cable. We've also had success using a cheap VGA to HDMI adaptor connected directly to the\nVGA output port.\n\nIn case of issues, use a proper VGA buffer / cable-driver like the AD8044. It's about 8 GBP though, so we did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"
- note removed: "VGA"
Changed lines of the file:
@@
 EESchema Schematic File Version 4
-LIBS:neotron-32-cache
-EELAYER 26 0
+EELAYER 30 0
 EELAYER END
 $Descr A4 11693 8268
@@
 F 2 "Connector_Dsub:DSUB-15-HD_Female_Horizontal_P2.29x1.98mm_EdgePinOffset3.03mm_Housed_MountingHolesOffset4.94mm" H 4600 3650 50  0001 C CNN
 F 3 "https://www.amphenol-icc.com/media/wysiwyg/files/drawing/c-cd-0012.pdf" H 4600 3650 50  0001 C CNN
-F 5 "Amphenol" H 5550 3250 50  0001 C CNN "Manufacturer"
-F 6 "ICD15S13E4GV00LF" H 5550 3250 50  0001 C CNN "PartNo"
+F 4 "Amphenol" H 5550 3250 50  0001 C CNN "Manufacturer"
+F 5 "ICD15S13E4GV00LF" H 5550 3250 50  0001 C CNN "PartNo"
 	1    5550 3250
 	1    0    0    -1
@@
 Wire Wire Line
 	5200 3650 5200 4000
-Text Notes 5500 2000 0    100  ~ 20
-VGA
+Text Notes 550  7700 0    50   Italic 0
+The VGA output is driven directly from the GPIO pins using a resistive divider. The output impedance is therefore all wrong. Best results\nare with an LCD monitor and a short VGA cable. We've also had success using a cheap VGA to HDMI adaptor connected directly to the\nVGA output port.\n\nIn case of issues, use a proper VGA buffer / cable-driver like the AD8044. It's about 8 GBP though, so we didn't bother.
 $EndSCHEMATC
