File: parallel.sch (KiCad schematic (older format))
At the start: 11 parts, among them J11 Conn_02x13_Top_Bottom, U5 MCP23S17_SP

Commit message: Adding MPNs.
Parts:
- U5: Manufacturer (none) -> Microchip; PartNo (none) -> MCP23S17-E/SP
Changed lines of the file:
@@
 F 2 "Package_DIP:DIP-28_W7.62mm" H 3650 2500 50  0001 L CNN
 F 3 "http://ww1.microchip.com/downloads/en/DeviceDoc/20001952C.pdf" H 3650 2400 50  0001 L CNN
+F 4 "Microchip" H 3450 3500 50  0001 C CNN "Manufacturer"
+F 5 "MCP23S17-E/SP" H 3450 3500 50  0001 C CNN "PartNo"
 	1    3450 3500
 	1    0    0    -1

Commit message: Updated BOM.
Parts:
- C10: Manufacturer (none) -> Vishay; PartNo (none) -> K104K15X7RF5TL2
- C11, C12, C13, C14, C15, C16, C17, C18: Manufacturer (none) -> Vishay; PartNo (none) -> K223K15X7RF5TL2
Changed lines of the file:
@@
 F 2 "Capacitor_THT:C_Disc_D3.0mm_W2.0mm_P2.50mm" H 8138 2650 50  0001 C CNN
 F 3 "~" H 8100 2800 50  0001 C CNN
+F 4 "Vishay" H 0   0   50  0001 C CNN "Manufacturer"
+F 5 "K223K15X7RF5TL2" H 0   0   50  0001 C CNN "PartNo"
 	1    8100 2800
 	0    1    1    0
@@
 F 2 "Capacitor_THT:C_Disc_D3.0mm_W2.0mm_P2.50mm" H 8138 4050 50  0001 C CNN
 F 3 "~" H 8100 4200 50  0001 C CNN
+F 4 "Vishay" H 0   0   50  0001 C CNN "Manufacturer"
+F 5 "K223K15X7RF5TL2" H 0   0   50  0001 C CNN "PartNo"
 	1    8100 4200
 	0    1    1    0
@@
 F 2 "Capacitor_THT:C_Disc_D3.0mm_W2.0mm_P2.50mm" H 8138 2850 50  0001 C CNN
 F 3 "~" H 8100 3000 50  0001 C CNN
+F 4 "Vishay" H 0   0   50  0001 C CNN "Manufacturer"
+F 5 "K223K15X7RF5TL2" H 0   0   50  0001 C CNN "PartNo"
 	1    8100 3000
 	0    1    1    0
@@
 F 2 "Capacitor_THT:C_Disc_D3.0mm_W2.0mm_P2.50mm" H 8138 3050 50  0001 C CNN
 F 3 "~" H 8100 3200 50  0001 C CNN
+F 4 "Vishay" H 0   0   50  0001 C CNN "Manufacturer"
+F 5 "K223K15X7RF5TL2" H 0   0   50  0001 C CNN "PartNo"
 	1    8100 3200
 	0    1    1    0
@@
 F 2 "Capacitor_THT:C_Disc_D3.0mm_W2.0mm_P2.50mm" H 8138 3250 50  0001 C CNN
 F 3 "~" H 8100 3400 50  0001 C CNN
+F 4 "Vishay" H 0   0   50  0001 C CNN "Manufacturer"
+F 5 "K223K15X7RF5TL2" H 0   0   50  0001 C CNN "PartNo"
 	1    8100 3400
 	0    1    1    0
@@
 F 2 "Capacitor_THT:C_Disc_D3.0mm_W2.0mm_P2.50mm" H 8138 3850 50  0001 C CNN
 F 3 "~" H 8100 4000 50  0001 C CNN
+F 4 "Vishay" H 0   0   50  0001 C CNN "Manufacturer"
+F 5 "K223K15X7RF5TL2" H 0   0   50  0001 C CNN "PartNo"
 	1    8100 4000
 	0    1    1    0
@@
 F 2 "Capacitor_THT:C_Disc_D3.0mm_W2.0mm_P2.50mm" H 8138 3650 50  0001 C CNN
 F 3 "~" H 8100 3800 50  0001 C CNN
+F 4 "Vishay" H 0   0   50  0001 C CNN "Manufacturer"
+F 5 "K223K15X7RF5TL2" H 0   0   50  0001 C CNN "PartNo"
 	1    8100 3800
 	0    1    1    0
@@
 F 2 "Capacitor_THT:C_Disc_D3.0mm_W2.0mm_P2.50mm" H 8138 3450 50  0001 C CNN
 F 3 "~" H 8100 3600 50  0001 C CNN
+F 4 "Vishay" H 0   0   50  0001 C CNN "Manufacturer"
+F 5 "K223K15X7RF5TL2" H 0   0   50  0001 C CNN "PartNo"
 	1    8100 3600
 	0    1    1    0
@@
 F 2 "Capacitor_THT:C_Disc_D3.0mm_W2.0mm_P2.50mm" H 1488 3300 50  0001 C CNN
 F 3 "~" H 1450 3450 50  0001 C CNN
+F 4 "Vishay" H 0   0   50  0001 C CNN "Manufacturer"
+F 5 "K104K15X7RF5TL2" H 0   0   50  0001 C CNN "PartNo"
 	1    1450 3450
 	1    0    0    -1
@@
 F 2 "Connector_PinHeader_2.54mm:PinHeader_2x13_P2.54mm_Vertical" H 6400 3650 50  0001 C CNN
 F 3 "~" H 6400 3650 50  0001 C CNN
+F 4 "~" H 0   0   50  0001 C CNN "Manufacturer"
+F 5 "~" H 0   0   50  0001 C CNN "PartNo"
 	1    6400 3650
 	1    0    0    -1

Commit message: Add some extra explanatory notes.
Other:
- note added: "Provides an 25-pin Parallel Port as found on an IBM PC. Implementation of SPP, EPP or ECP is down to the software on the MCU, as this is a\nbasic 3.3v SPI to GPIO convertor chip.\n\nThe strobe signal is direct from the CPU to allow it to be toggled on and off relatively quickly. The MCP23S17 can be configured to generate\ninputs to avoid the CPU busy-waiting for ACK from the remote device.\n\nIf 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"
- note removed: "Parallel Printer Port"
Changed lines of the file:
@@
 EESchema Schematic File Version 4
-LIBS:neotron-32-cache
-EELAYER 26 0
+EELAYER 30 0
 EELAYER END
 $Descr A4 11693 8268
@@
 Text Label 4250 3400 0    50   ~ 0
 ~SELPRI
-Text Notes 4850 1850 0    100  ~ 20
-Parallel Printer Port
 Wire Bus Line
 	7200 3150 7200 4550
@@
 Wire Bus Line
 	4800 2400 4800 4550
+Text Notes 550  7700 0    50   Italic 0
+Provides an 25-pin Parallel Port as found on an IBM PC. Implementation of SPP, EPP or ECP is down to the software on the MCU, as this is a\nbasic 3.3v SPI to GPIO convertor chip.\n\nThe strobe signal is direct from the CPU to allow it to be toggled on and off relatively quickly. The MCP23S17 can be configured to generate\ninputs to avoid the CPU busy-waiting for ACK from the remote device.\n\nIf you want a proper DB25 Parallel port, you will need a 26-way IDC ribbon to DB25 male cable. These were commonly fitted to PCs in the\n1990s as the ISA I/O expansion cards and/or motherboards of the time often didn't have room for all of the ports on the backplate. We\ndidn't fit a DB25 to this board due to similar space issues.
 $EndSCHEMATC

Commit message: Moved non-standard components into local libraries.
neotron-32.lib is the symbol library.
neotron-32.pretty is the footprint library.

Also swapped the DE9 and DB25 headers for IDC boxed versions. Involved
moving a resistor out of the way.

The Keystone 103 battery holder is a straight copy of the standard
footprint, but with the Courtyard removed to bypass the 'Courtyard is
not closed' DRC error.
Parts:
- J11: footprint Connector_PinHeader_2.54mm:PinHeader_2x13_P2.54mm_Vertical -> Connector_IDC:IDC-Header_2x13_P2.54mm_Vertical
Changed lines of the file:
@@
 F 0 "J11" H 6450 4467 50  0000 C CNN
 F 1 "Conn_02x13_Top_Bottom" H 6450 4376 50  0000 C CNN
-F 2 "Connector_PinHeader_2.54mm:PinHeader_2x13_P2.54mm_Vertical" H 6400 3650 50  0001 C CNN
+F 2 "Connector_IDC:IDC-Header_2x13_P2.54mm_Vertical" H 6400 3650 50  0001 C CNN
 F 3 "~" H 6400 3650 50  0001 C CNN
 F 4 "~" H 0   0   50  0001 C CNN "Manufacturer"
@@
 Text Label 4250 3400 0    50   ~ 0
 ~SELPRI
+Text Notes 550  7700 0    50   Italic 0
+Provides an 25-pin Parallel Port as found on an IBM PC. Implementation of SPP, EPP or ECP is down to the software on the MCU, as this is a\nbasic 3.3v SPI to GPIO convertor chip.\n\nThe strobe signal is direct from the CPU to allow it to be toggled on and off relatively quickly. The MCP23S17 can be configured to generate\ninputs to avoid the CPU busy-waiting for ACK from the remote device.\n\nIf you want a proper DB25 Parallel port, you will need a 26-way IDC ribbon to DB25 male cable. These were commonly fitted to PCs in the\n1990s as the ISA I/O expansion cards and/or motherboards of the time often didn't have room for all of the ports on the backplate. We\ndidn't fit a DB25 to this board due to similar space issues.
 Wire Bus Line
 	7200 3150 7200 4550
@@
 Wire Bus Line
 	4800 2400 4800 4550
-Text Notes 550  7700 0    50   Italic 0
-Provides an 25-pin Parallel Port as found on an IBM PC. Implementation of SPP, EPP or ECP is down to the software on the MCU, as this is a\nbasic 3.3v SPI to GPIO convertor chip.\n\nThe strobe signal is direct from the CPU to allow it to be toggled on and off relatively quickly. The MCP23S17 can be configured to generate\ninputs to avoid the CPU busy-waiting for ACK from the remote device.\n\nIf you want a proper DB25 Parallel port, you will need a 26-way IDC ribbon to DB25 male cable. These were commonly fitted to PCs in the\n1990s as the ISA I/O expansion cards and/or motherboards of the time often didn't have room for all of the ports on the backplate. We\ndidn't fit a DB25 to this board due to similar space issues.
 $EndSCHEMATC

Commit message: Fixed footprints.
) Parallel port was wrongly numbered.
) Input fuse has 0.2" leg spacing.
) Also cleaned up a few more diagonals.
Parts:
- J11: value Conn_02x13_Top_Bottom -> Conn_02x13_Header; symbol Connector_Generic:Conn_02x13_Top_Bottom -> Connector_Generic:Conn_02x13_Odd_Even
Connections:
- net ACK: now also J11.19 (Pin_19); no longer J11.10 (Pin_10)
- net D0: now also J11.3 (Pin_3); no longer J11.2 (Pin_2)
- net D1: now also J11.5 (Pin_5); no longer J11.3 (Pin_3)
- net D2: now also J11.7 (Pin_7); no longer J11.4 (Pin_4)
- net D3: now also J11.9 (Pin_9); no longer J11.5 (Pin_5)
- net D4: now also J11.11 (Pin_11); no longer J11.6 (Pin_6)
- net D5: now also J11.13 (Pin_13); no longer J11.7 (Pin_7)
- net D6: now also J11.15 (Pin_15); no longer J11.8 (Pin_8)
- net D7: now also J11.17 (Pin_17); no longer J11.9 (Pin_9)
- net ERROR: now also J11.4 (Pin_4); no longer J11.15 (Pin_15)
- net GND: now also J11.10 (Pin_10), J11.12 (Pin_12), J11.14 (Pin_14), J11.16 (Pin_16); no longer J11.19 (Pin_19), J11.21 (Pin_21), J11.23 (Pin_23), J11.25 (Pin_25)
- net POUT: now also J11.23 (Pin_23); no longer J11.12 (Pin_12)
- net RESET: now also J11.6 (Pin_6); no longer J11.16 (Pin_16)
- net SELECT: now also J11.25 (Pin_25); no longer J11.13 (Pin_13)
- net ~BUSY: now also J11.21 (Pin_21); no longer J11.11 (Pin_11)
- net ~LF: now also J11.2 (Pin_2); no longer J11.14 (Pin_14)
- net ~SELPRI: now also J11.8 (Pin_8); no longer J11.17 (Pin_17)
Changed lines of the file:
@@
 	1450 3600 1450 3700
 $Comp
-L Connector_Generic:Conn_02x13_Top_Bottom J11
+L Connector_Generic:Conn_02x13_Odd_Even J11
 U 1 1 5DF553E8
 P 6400 3650
 F 0 "J11" H 6450 4467 50  0000 C CNN
-F 1 "Conn_02x13_Top_Bottom" H 6450 4376 50  0000 C CNN
+F 1 "Conn_02x13_Header" H 6450 4376 50  0000 C CNN
 F 2 "Connector_IDC:IDC-Header_2x13_P2.54mm_Vertical" H 6400 3650 50  0001 C CNN
 F 3 "~" H 6400 3650 50  0001 C CNN
