File: serial.sch (KiCad schematic (older format))
At the start: 7 parts, among them J18 Conn_02x05, U8 ICL3232CPZMAX

Commit message: Replace PartNum with MPN so Kicost can see it.
Parts:
- C24, C25: PartNo K104K15X7RF5TL2 -> (none); mpn (none) -> K104K15X7RF5TL2
- C26, C27, C28: PartNo K474Z20Y5VE5TL2 -> (none); mpn (none) -> K474Z20Y5VE5TL2
- J18: PartNo M20-9760546 -> (none); mpn (none) -> M20-9760546
- U8: PartNo ICL3232CPZ -> (none); mpn (none) -> ICL3232CPZ
Changed lines of the file:
@@
 F 3 "https://www.renesas.com/en-us/www/doc/datasheet/hin232-36-37-38-39-40-41.pdf" H 5600 3750 50  0001 C CNN
 F 4 "Renesas" H 5600 3650 50  0001 C CNN "Manufacturer"
-F 5 "ICL3232CPZ" H 5600 3650 50  0001 C CNN "PartNo"
+F 5 "ICL3232CPZ" H 5600 3650 50  0001 C CNN "mpn"
 	1    5600 3650
 	1    0    0    -1
@@
 F 3 "~" H 6500 2900 50  0001 C CNN
 F 4 "Vishay" H 0   0   50  0001 C CNN "Manufacturer"
-F 5 "K474Z20Y5VE5TL2" H 0   0   50  0001 C CNN "PartNo"
+F 5 "K474Z20Y5VE5TL2" H 0   0   50  0001 C CNN "mpn"
 	1    6500 2900
 	1    0    0    -1
@@
 F 3 "~" H 6800 3550 50  0001 C CNN
 F 4 "Vishay" H 0   0   50  0001 C CNN "Manufacturer"
-F 5 "K474Z20Y5VE5TL2" H 0   0   50  0001 C CNN "PartNo"
+F 5 "K474Z20Y5VE5TL2" H 0   0   50  0001 C CNN "mpn"
 	1    6800 3550
 	0    1    1    0
@@
 F 3 "~" H 4650 2900 50  0001 C CNN
 F 4 "Vishay" H 0   0   50  0001 C CNN "Manufacturer"
-F 5 "K104K15X7RF5TL2" H 0   0   50  0001 C CNN "PartNo"
+F 5 "K104K15X7RF5TL2" H 0   0   50  0001 C CNN "mpn"
 	1    4650 2900
 	-1   0    0    1
@@
 F 3 "~" H 3350 3100 50  0001 C CNN
 F 4 "Vishay" H 0   0   50  0001 C CNN "Manufacturer"
-F 5 "K104K15X7RF5TL2" H 0   0   50  0001 C CNN "PartNo"
+F 5 "K104K15X7RF5TL2" H 0   0   50  0001 C CNN "mpn"
 	1    3350 3100
 	-1   0    0    1
@@
 F 3 "~" H 7050 2800 50  0001 C CNN
 F 4 "Vishay" H 0   0   50  0001 C CNN "Manufacturer"
-F 5 "K474Z20Y5VE5TL2" H 0   0   50  0001 C CNN "PartNo"
+F 5 "K474Z20Y5VE5TL2" H 0   0   50  0001 C CNN "mpn"
 	1    7050 2800
 	1    0    0    -1
@@
 F 3 "~" H 8100 4050 50  0001 C CNN
 F 4 "Harwin" H 8100 4050 50  0001 C CNN "Manufacturer"
-F 5 "M20-9760546" H 8100 4050 50  0001 C CNN "PartNo"
+F 5 "M20-9760546" H 8100 4050 50  0001 C CNN "mpn"
 	1    8100 4050
 	1    0    0    1

Commit message: Tweaks to the BOM.
Marking parts as DNP=1 should stop them appearing in the BOM.
Also set multi-parts for ICs in sockets.
Parts:
- C24, C25, C26, C27, C28: DNP (none) -> 0
- J18: DNP (none) -> 0; Manufacturer Harwin -> On Shore Technology; mpn M20-9760546 -> 302-S101
- U8: DNP (none) -> 0; Manufacturer Renesas -> Renesas;On Shore Technology; mpn ICL3232CPZ -> ICL3232CPZ;ED16DT
Changed lines of the file:
@@
 F 2 "Package_DIP:DIP-16_W7.62mm" H 5650 2600 50  0001 L CNN
 F 3 "https://www.renesas.com/en-us/www/doc/datasheet/hin232-36-37-38-39-40-41.pdf" H 5600 3750 50  0001 C CNN
-F 4 "Renesas" H 5600 3650 50  0001 C CNN "Manufacturer"
-F 5 "ICL3232CPZ" H 5600 3650 50  0001 C CNN "mpn"
+F 4 "Renesas;On Shore Technology" H 5600 3650 50  0001 C CNN "Manufacturer"
+F 5 "ICL3232CPZ;ED16DT" H 5600 3650 50  0001 C CNN "mpn"
+F 6 "0" H 5600 3650 50  0001 C CNN "DNP"
 	1    5600 3650
 	1    0    0    -1
@@
 F 4 "Vishay" H 0   0   50  0001 C CNN "Manufacturer"
 F 5 "K474Z20Y5VE5TL2" H 0   0   50  0001 C CNN "mpn"
+F 6 "0" H 6500 2900 50  0001 C CNN "DNP"
 	1    6500 2900
 	1    0    0    -1
@@
 F 4 "Vishay" H 0   0   50  0001 C CNN "Manufacturer"
 F 5 "K474Z20Y5VE5TL2" H 0   0   50  0001 C CNN "mpn"
+F 6 "0" H 6800 3550 50  0001 C CNN "DNP"
 	1    6800 3550
 	0    1    1    0
@@
 F 4 "Vishay" H 0   0   50  0001 C CNN "Manufacturer"
 F 5 "K104K15X7RF5TL2" H 0   0   50  0001 C CNN "mpn"
+F 6 "0" H 4650 2900 50  0001 C CNN "DNP"
 	1    4650 2900
 	-1   0    0    1
@@
 F 4 "Vishay" H 0   0   50  0001 C CNN "Manufacturer"
 F 5 "K104K15X7RF5TL2" H 0   0   50  0001 C CNN "mpn"
+F 6 "0" H 3350 3100 50  0001 C CNN "DNP"
 	1    3350 3100
 	-1   0    0    1
@@
 F 4 "Vishay" H 0   0   50  0001 C CNN "Manufacturer"
 F 5 "K474Z20Y5VE5TL2" H 0   0   50  0001 C CNN "mpn"
+F 6 "0" H 7050 2800 50  0001 C CNN "DNP"
 	1    7050 2800
 	1    0    0    -1
@@
 F 2 "Connector_IDC:IDC-Header_2x05_P2.54mm_Vertical" H 8100 4050 50  0001 C CNN
 F 3 "~" H 8100 4050 50  0001 C CNN
-F 4 "Harwin" H 8100 4050 50  0001 C CNN "Manufacturer"
-F 5 "M20-9760546" H 8100 4050 50  0001 C CNN "mpn"
+F 4 "On Shore Technology" H 8100 4050 50  0001 C CNN "Manufacturer"
+F 5 "302-S101" H 8100 4050 50  0001 C CNN "mpn"
+F 6 "0" H 8100 4050 50  0001 C CNN "DNP"
 	1    8100 4050
 	1    0    0    1
