File: Kicad/parallel.sch (KiCad schematic (older format))
At the start: 11 parts, among them J601 Conn_02x13_Header, U601 MCP23S17_SP

Commit message: Working on layout.
Laid out the parallel port - reordered some pins to make it easier.
Set the minimum track widths to 6 mil/6 mil with a 6mm/3mm via.
Replaced the SPST power switch with a PUE to match the reset switch.
Attached some existing 3D models to the PCB footprints.
Connections:
- net ACK: now also U601.4 (GPB3); no longer U601.1 (GPB0)
- net ERROR: now also U601.7 (GPB6); no longer U601.6 (GPB5)
- net POUT: now also U601.2 (GPB1); no longer U601.3 (GPB2)
- net RESET: now also U601.6 (GPB5); no longer U601.7 (GPB6)
- net SELECT: now also U601.1 (GPB0); no longer U601.4 (GPB3)
- net ~BUSY: now also U601.3 (GPB2); no longer U601.2 (GPB1)
- net ~LF: now also U601.8 (GPB7); no longer U601.5 (GPB4)
- net ~SELPRI: now also U601.5 (GPB4); no longer U601.8 (GPB7)
Changed lines of the file:
@@
 	1    0    0    -1
 $EndComp
+Text Label 4250 3000 0    50   ~ 0
+ACK
+Text Label 4250 2900 0    50   ~ 0
+~BUSY
+Text Label 4250 2800 0    50   ~ 0
+POUT
 Text Label 4250 2700 0    50   ~ 0
-ACK
-Text Label 4250 2800 0    50   ~ 0
-~BUSY
-Text Label 4250 2900 0    50   ~ 0
-POUT
-Text Label 4250 3000 0    50   ~ 0
 SELECT
 Text Label 7900 4200 2    50   ~ 0
@@
 Text Notes 1200 4100 0    50   ~ 0
 Fit close to Vdd
+Text Label 4250 3400 0    50   ~ 0
+~LF
+Text Label 4250 3300 0    50   ~ 0
+ERROR
+Text Label 4250 3200 0    50   ~ 0
+RESET
 Text Label 4250 3100 0    50   ~ 0
-~LF
-Text Label 4250 3200 0    50   ~ 0
-ERROR
-Text Label 4250 3300 0    50   ~ 0
-RESET
-Text Label 4250 3400 0    50   ~ 0
 ~SELPRI
 Text Notes 550  7700 0    50   Italic 0
