File: Kicad/serial.sch (KiCad schematic (older format))
At the start: 7 parts, among them J1001 Conn_02x05, U1001 ICL3232CPZMAX

Commit message: Switch to 1598D enclosure.
Use MIC2005A current limiter on input.
Use soft on/off switch from Atmega.
Atmega connects to Tiva over I2C.
Use full-size SD card.
Parts:
- renumbered C1001 to C901, C1002 to C902, C1003 to C903, C1004 to C904, C1005 to C905, J1001 to J901, U1001 to U901
Changed lines of the file:
@@
 $Descr A4 11693 8268
 encoding utf-8
-Sheet 10 10
+Sheet 9 12
 Title "Neotron 32K Main PCB"
 Date "2020-03-29"
@@
 RS232_CTS_TO_MCU
 $Comp
-L Interface_UART:MAX232 U1001
+L Interface_UART:MAX232 U901
 U 1 1 5E0F5F91
 P 5600 3650
-F 0 "U1001" H 6100 4750 50  0000 C CNN
+F 0 "U901" H 6100 4750 50  0000 C CNN
 F 1 "ICL3232CPZMAX" H 5150 4750 50  0000 C CNN
 F 2 "Package_DIP:DIP-16_W7.62mm" H 5650 2600 50  0001 L CNN
@@
 	7300 3450 7300 3400
 $Comp
-L Device:C C1003
+L Device:C C903
 U 1 1 5E181E57
 P 6500 2900
-F 0 "C1003" H 6615 2946 50  0000 L CNN
+F 0 "C903" H 6615 2946 50  0000 L CNN
 F 1 "100n" H 6615 2855 50  0000 L CNN
 F 2 "Capacitor_THT:C_Disc_D3.0mm_W2.0mm_P2.50mm" H 6538 2750 50  0001 C CNN
@@
 $EndComp
 $Comp
-L Device:C C1004
+L Device:C C904
 U 1 1 5E182C3F
 P 6800 3550
-F 0 "C1004" V 6650 3450 50  0000 C CNN
+F 0 "C904" V 6650 3450 50  0000 C CNN
 F 1 "100n" V 6650 3650 50  0000 C CNN
 F 2 "Capacitor_THT:C_Disc_D3.0mm_W2.0mm_P2.50mm" H 6838 3400 50  0001 C CNN
@@
 $EndComp
 $Comp
-L Device:C C1002
+L Device:C C902
 U 1 1 5E182DBA
 P 4650 2900
-F 0 "C1002" H 4900 2850 50  0000 R CNN
+F 0 "C902" H 4900 2850 50  0000 R CNN
 F 1 "100n" H 4950 2950 50  0000 R CNN
 F 2 "Capacitor_THT:C_Disc_D3.0mm_W2.0mm_P2.50mm" H 4688 2750 50  0001 C CNN
@@
 $EndComp
 $Comp
-L Device:C C1001
+L Device:C C901
 U 1 1 5E183108
 P 3350 3100
-F 0 "C1001" H 3235 3054 50  0000 R CNN
+F 0 "C901" H 3235 3054 50  0000 R CNN
 F 1 "100n" H 3235 3145 50  0000 R CNN
 F 2 "Capacitor_THT:C_Disc_D3.0mm_W2.0mm_P2.50mm" H 3388 2950 50  0001 C CNN
@@
 	4650 3050 4800 3050
 $Comp
-L Device:C C1005
+L Device:C C905
 U 1 1 5E188858
 P 7050 2800
-F 0 "C1005" H 7165 2846 50  0000 L CNN
+F 0 "C905" H 7165 2846 50  0000 L CNN
 F 1 "100n" H 7165 2755 50  0000 L CNN
 F 2 "Capacitor_THT:C_Disc_D3.0mm_W2.0mm_P2.50mm" H 7088 2650 50  0001 C CNN
@@
 NoConn ~ 8400 3950
 $Comp
-L Connector_Generic:Conn_02x05_Top_Bottom J1001
+L Connector_Generic:Conn_02x05_Top_Bottom J901
 U 1 1 5E02DBC9
 P 8100 4050
-F 0 "J1001" H 8150 3625 50  0000 C CNN
+F 0 "J901" H 8150 3625 50  0000 C CNN
 F 1 "Conn_02x05" H 8150 3716 50  0000 C CNN
 F 2 "Connector_IDC:IDC-Header_2x05_P2.54mm_Vertical" H 8100 4050 50  0001 C CNN
